Commit message: Converted valkyries A-E to use generic macro

File: model/robots/valkyrie_A.xacro (robot description, xacro)
@@ -1,4 +1,5 @@
 <?xml version="1.0" ?>
 <robot xmlns:xacro="http://www.ros.org/wiki/xacro" name="ValkyrieA">
+    <xacro:property name="robot_type_suffix" value=""/>
     <xacro:include filename="./valkyrie_generic.xacro"/>
     <xacro:valkyrie_generic suffix="A"/>

File: model/robots/valkyrie_A_arm_mass_sims.xacro (robot description, xacro)
@@ -1,27 +1,6 @@
+<?xml version="1.0" ?>
 <robot xmlns:xacro="http://www.ros.org/wiki/xacro" name="valkyrie">
-	<xacro:property name="leg_mesh_dir" value="package://val_description/model/meshes/legs"/>
-    <xacro:property name="arm_mesh_dir" value="package://val_description/model/meshes/arms"/>
-    <xacro:property name="waist_mesh_dir" value="package://val_description/model/meshes/torso"/>
-    <xacro:property name="head_mesh_dir" value="package://val_description/model/meshes/head"/>
-    <xacro:property name="pelvis_mesh_dir" value="package://val_description/model/meshes/pelvis"/>
-    <xacro:property name="fingers_mesh_dir" value="package://val_description/model/meshes/fingers"/>
-    <xacro:property name="robot_type_suffix" value="_sim"/>
-    <xacro:include filename="../../model/robots/common/xacro/generic_models.xacro" />
-    <xacro:include filename="../../common/xacro/nodes/valkyrie_nodes.xacro"/>
-    <xacro:include filename="../../model/robots/common/xacro/sensors/sensor_transforms.xacro"/>
-    <xacro:include filename="../../model/robots/common/xacro/config/valkyrie_A_transmissions.xacro" />
-    <xacro:include filename="../../common/xacro/serial_numbers/valkyrie_A_serials.xacro"/>
-    <xacro:include filename="../../common/xacro/api/valkyrie_A_api.xacro"/>
-    <xacro:include filename="../../common/xacro/dev_ports/valkyrie_A_ports.xacro"/>
-    <!-- Pelvis include -->
-    <xacro:include filename="../../model/robots/common/xacro/pelvis/pelvis_includes.xacro"/>
-    <!-- Leg include -->
-    <xacro:include filename="../../model/robots/common/xacro/leg/leg_includes.xacro"/>
-    <!-- Head include -->
-    <xacro:include filename="../../model/robots/common/xacro/head/head_includes.xacro"/>
-    <!-- Arm include -->
-    <xacro:include filename="../../model/robots/common/xacro/arm/arm_includes.xacro"/>
-    <!-- Waist include -->
-    <xacro:include filename="../../model/robots/common/xacro/waist/waist_includes.xacro"/>
-    <xacro:include filename="../../model/robots/common/xacro/valkyrie_arm_mass_sims_base_hw.xacro"/>
+	<xacro:property name="robot_type_suffix" value="_sim"/>
+    <xacro:include filename="./valkyrie_generic.xacro"/>
+    <xacro:valkyrie_generic suffix="A"/>
 </robot>

File: model/robots/valkyrie_B.xacro (robot description, xacro)
@@ -1,28 +1,6 @@
-<robot xmlns:xacro="http://www.ros.org/wiki/xacro" name="ValkyrieB">
-	<xacro:property name="leg_mesh_dir" value="package://val_description/model/meshes/legs"/>
-    <xacro:property name="arm_mesh_dir" value="package://val_description/model/meshes/arms"/>
-    <xacro:property name="waist_mesh_dir" value="package://val_description/model/meshes/torso"/>
-    <xacro:property name="head_mesh_dir" value="package://val_description/model/meshes/head"/>
-    <xacro:property name="pelvis_mesh_dir" value="package://val_description/model/meshes/pelvis"/>
-    <xacro:property name="fingers_mesh_dir" value="package://val_description/model/meshes/fingers"/>
-    <xacro:property name="robot_type_suffix" value=""/>
-	<xacro:include filename="../../model/robots/common/xacro/generic_models.xacro" />
-    <xacro:include filename="../../common/xacro/nodes/valkyrie_nodes.xacro"/>
-    <xacro:include filename="../../model/robots/common/xacro/sensors/sensor_transforms.xacro"/>
-    <xacro:include filename="../../model/robots/common/xacro/config/valkyrie_B_transmissions.xacro" />
-	<xacro:include filename="../../common/xacro/serial_numbers/valkyrie_B_serials.xacro"/>
-    <xacro:include filename="../../common/xacro/api/valkyrie_B_api.xacro"/>
-    <xacro:include filename="../../common/xacro/dev_ports/valkyrie_B_ports.xacro"/>
-    <xacro:include filename="../../model/robots/common/xacro/common_bodies.xacro" />
-    <!-- Pelvis include -->
-    <xacro:include filename="../../model/robots/common/xacro/pelvis/pelvis_includes.xacro"/>
-    <!-- Leg include -->
-    <xacro:include filename="../../model/robots/common/xacro/leg/leg_includes.xacro"/>
-    <!-- Head include -->
-    <xacro:include filename="../../model/robots/common/xacro/head/head_includes.xacro"/>
-    <!-- Arm include -->
-    <xacro:include filename="../../model/robots/common/xacro/arm/arm_includes.xacro"/>
-    <!-- Waist include -->
-    <xacro:include filename="../../model/robots/common/xacro/waist/waist_includes.xacro"/>
-    <xacro:include filename="../../model/robots/common/xacro/valkyrie_base_hw.xacro"/>
+<?xml version="1.0" ?>
+<robot xmlns:xacro="http://www.ros.org/wiki/xacro" name="valkyrie">
+	<xacro:property name="robot_type_suffix" value=""/>
+    <xacro:include filename="./valkyrie_generic.xacro"/>
+    <xacro:valkyrie_generic suffix="B"/>
 </robot>

File: model/robots/valkyrie_B_arm_mass_sims.xacro (robot description, xacro)
@@ -1,27 +1,6 @@
+<?xml version="1.0" ?>
 <robot xmlns:xacro="http://www.ros.org/wiki/xacro" name="valkyrie">
-	<xacro:property name="leg_mesh_dir" value="package://val_description/model/meshes/legs"/>
-    <xacro:property name="arm_mesh_dir" value="package://val_description/model/meshes/arms"/>
-    <xacro:property name="waist_mesh_dir" value="package://val_description/model/meshes/torso"/>
-    <xacro:property name="head_mesh_dir" value="package://val_description/model/meshes/head"/>
-    <xacro:property name="pelvis_mesh_dir" value="package://val_description/model/meshes/pelvis"/>
-    <xacro:property name="fingers_mesh_dir" value="package://val_description/model/meshes/fingers"/>
-    <xacro:property name="robot_type_suffix" value="_sim"/>
-    <xacro:include filename="../../model/robots/common/xacro/generic_models.xacro" />
-    <xacro:include filename="../../common/xacro/nodes/valkyrie_nodes.xacro"/>
-    <xacro:include filename="../../model/robots/common/xacro/sensors/sensor_transforms.xacro"/>
-    <xacro:include filename="../../model/robots/common/xacro/config/valkyrie_B_transmissions.xacro"/>
-    <xacro:include filename="../../common/xacro/serial_numbers/valkyrie_B_serials.xacro"/>
-    <xacro:include filename="../../common/xacro/api/valkyrie_B_api.xacro"/>
-    <xacro:include filename="../../common/xacro/dev_ports/valkyrie_B_ports.xacro"/>
-    <!-- Pelvis include -->
-    <xacro:include filename="../../model/robots/common/xacro/pelvis/pelvis_includes.xacro"/>
-    <!-- Leg include -->
-    <xacro:include filename="../../model/robots/common/xacro/leg/leg_includes.xacro"/>
-    <!-- Head include -->
-    <xacro:include filename="../../model/robots/common/xacro/head/head_includes.xacro"/>
-    <!-- Arm include -->
-    <xacro:include filename="../../model/robots/common/xacro/arm/arm_includes.xacro"/>
-    <!-- Waist include -->
-    <xacro:include filename="../../model/robots/common/xacro/waist/waist_includes.xacro"/>
-    <xacro:include filename="../../model/robots/common/xacro/valkyrie_arm_mass_sims_base_hw.xacro"/>
+	<xacro:property name="robot_type_suffix" value="_sim"/>
+    <xacro:include filename="./valkyrie_generic.xacro"/>
+    <xacro:valkyrie_generic suffix="B"/>
 </robot>

File: model/robots/valkyrie_C.xacro (robot description, xacro)
@@ -1,28 +1,6 @@
-<robot xmlns:xacro="http://www.ros.org/wiki/xacro" name="ValkyrieC">
-	<xacro:property name="leg_mesh_dir" value="package://val_description/model/meshes/legs"/>
-    <xacro:property name="arm_mesh_dir" value="package://val_description/model/meshes/arms"/>
-    <xacro:property name="waist_mesh_dir" value="package://val_description/model/meshes/torso"/>
-    <xacro:property name="head_mesh_dir" value="package://val_description/model/meshes/head"/>
-    <xacro:property name="pelvis_mesh_dir" value="package://val_description/model/meshes/pelvis"/>
-    <xacro:property name="fingers_mesh_dir" value="package://val_description/model/meshes/fingers"/>
-    <xacro:property name="robot_type_suffix" value=""/>
-	<xacro:include filename="../../model/robots/common/xacro/generic_models.xacro" />
-    <xacro:include filename="../../common/xacro/nodes/valkyrie_nodes.xacro"/>
-    <xacro:include filename="../../model/robots/common/xacro/sensors/sensor_transforms.xacro"/>
-    <xacro:include filename="../../model/robots/common/xacro/config/valkyrie_C_transmissions.xacro" />
-    <xacro:include filename="../../common/xacro/serial_numbers/valkyrie_C_serials.xacro"/>
-    <xacro:include filename="../../common/xacro/api/valkyrie_C_api.xacro"/>
-    <xacro:include filename="../../common/xacro/dev_ports/valkyrie_C_ports.xacro"/>
-    <xacro:include filename="../../model/robots/common/xacro/common_bodies.xacro" />
-    <!-- Pelvis include -->
-    <xacro:include filename="../../model/robots/common/xacro/pelvis/pelvis_includes.xacro"/>
-    <!-- Leg include -->
-    <xacro:include filename="../../model/robots/common/xacro/leg/leg_includes.xacro"/>
-    <!-- Head include -->
-    <xacro:include filename="../../model/robots/common/xacro/head/head_includes.xacro"/>
-    <!-- Arm include -->
-    <xacro:include filename="../../model/robots/common/xacro/arm/arm_includes.xacro"/>
-    <!-- Waist include -->
-    <xacro:include filename="../../model/robots/common/xacro/waist/waist_includes.xacro"/>
-    <xacro:include filename="../../model/robots/common/xacro/valkyrie_base_hw.xacro"/>
+<?xml version="1.0" ?>
+<robot xmlns:xacro="http://www.ros.org/wiki/xacro" name="valkyrie">
+	<xacro:property name="robot_type_suffix" value=""/>
+    <xacro:include filename="./valkyrie_generic.xacro"/>
+    <xacro:valkyrie_generic suffix="C"/>
 </robot>

File: model/robots/valkyrie_C_arm_mass_sims.xacro (robot description, xacro)
@@ -1,27 +1,6 @@
+<?xml version="1.0" ?>
 <robot xmlns:xacro="http://www.ros.org/wiki/xacro" name="valkyrie">
-	<xacro:property name="leg_mesh_dir" value="package://val_description/model/meshes/legs"/>
-    <xacro:property name="arm_mesh_dir" value="package://val_description/model/meshes/arms"/>
-    <xacro:property name="waist_mesh_dir" value="package://val_description/model/meshes/torso"/>
-    <xacro:property name="head_mesh_dir" value="package://val_description/model/meshes/head"/>
-    <xacro:property name="pelvis_mesh_dir" value="package://val_description/model/meshes/pelvis"/>
-    <xacro:property name="fingers_mesh_dir" value="package://val_description/model/meshes/fingers"/>
-    <xacro:property name="robot_type_suffix" value="_sim"/>
-    <xacro:include filename="../../model/robots/common/xacro/generic_models.xacro" />
-    <xacro:include filename="../../common/xacro/nodes/valkyrie_nodes.xacro"/>
-    <xacro:include filename="../../model/robots/common/xacro/sensors/sensor_transforms.xacro"/>
-    <xacro:include filename="../../model/robots/common/xacro/config/valkyrie_C_transmissions.xacro" />
-    <xacro:include filename="../../common/xacro/serial_numbers/valkyrie_C_serials.xacro"/>
-    <xacro:include filename="../../common/xacro/api/valkyrie_C_api.xacro"/>
-    <xacro:include filename="../../common/xacro/dev_ports/valkyrie_C_ports.xacro"/>
-    <!-- Pelvis include -->
-    <xacro:include filename="../../model/robots/common/xacro/pelvis/pelvis_includes.xacro"/>
-    <!-- Leg include -->
-    <xacro:include filename="../../model/robots/common/xacro/leg/leg_includes.xacro"/>
-    <!-- Head include -->
-    <xacro:include filename="../../model/robots/common/xacro/head/head_includes.xacro"/>
-    <!-- Arm include -->
-    <xacro:include filename="../../model/robots/common/xacro/arm/arm_includes.xacro"/>
-    <!-- Waist include -->
-    <xacro:include filename="../../model/robots/common/xacro/waist/waist_includes.xacro"/>
-    <xacro:include filename="../../model/robots/common/xacro/valkyrie_arm_mass_sims_base_hw.xacro"/>
+	<xacro:property name="robot_type_suffix" value="_sim"/>
+    <xacro:include filename="./valkyrie_generic.xacro"/>
+    <xacro:valkyrie_generic suffix="C"/>
 </robot>

File: model/robots/valkyrie_D.xacro (robot description, xacro)
@@ -1,28 +1,6 @@
-<robot xmlns:xacro="http://www.ros.org/wiki/xacro" name="ValkyrieD">
-	<xacro:property name="leg_mesh_dir" value="package://val_description/model/meshes/legs"/>
-    <xacro:property name="arm_mesh_dir" value="package://val_description/model/meshes/arms"/>
-    <xacro:property name="waist_mesh_dir" value="package://val_description/model/meshes/torso"/>
-    <xacro:property name="head_mesh_dir" value="package://val_description/model/meshes/head"/>
-    <xacro:property name="pelvis_mesh_dir" value="package://val_description/model/meshes/pelvis"/>
-    <xacro:property name="fingers_mesh_dir" value="package://val_description/model/meshes/fingers"/>
-    <xacro:property name="robot_type_suffix" value=""/>
-	<xacro:include filename="../../model/robots/common/xacro/generic_models.xacro" />
-    <xacro:include filename="../../common/xacro/nodes/valkyrie_nodes.xacro"/>
-    <xacro:include filename="../../model/robots/common/xacro/sensors/sensor_transforms.xacro"/>
-    <xacro:include filename="../../model/robots/common/xacro/config/valkyrie_D_transmissions.xacro" />
-    <xacro:include filename="../../common/xacro/serial_numbers/valkyrie_D_serials.xacro"/>
-    <xacro:include filename="../../common/xacro/api/valkyrie_D_api.xacro"/>
-    <xacro:include filename="../../common/xacro/dev_ports/valkyrie_D_ports.xacro"/>
-    <xacro:include filename="../../model/robots/common/xacro/common_bodies.xacro" />
-    <!-- Pelvis include -->
-    <xacro:include filename="../../model/robots/common/xacro/pelvis/pelvis_includes.xacro"/>
-    <!-- Leg include -->
-    <xacro:include filename="../../model/robots/common/xacro/leg/leg_includes.xacro"/>
-    <!-- Head include -->
-    <xacro:include filename="../../model/robots/common/xacro/head/head_includes.xacro"/>
-    <!-- Arm include -->
-    <xacro:include filename="../../model/robots/common/xacro/arm/arm_includes.xacro"/>
-    <!-- Waist include -->
-    <xacro:include filename="../../model/robots/common/xacro/waist/waist_includes.xacro"/>
-    <xacro:include filename="../../model/robots/common/xacro/valkyrie_base_hw.xacro"/>
+<?xml version="1.0" ?>
+<robot xmlns:xacro="http://www.ros.org/wiki/xacro" name="valkyrie">
+	<xacro:property name="robot_type_suffix" value=""/>
+    <xacro:include filename="./valkyrie_generic.xacro"/>
+    <xacro:valkyrie_generic suffix="D"/>
 </robot>

File: model/robots/valkyrie_D_arm_mass_sims.xacro (robot description, xacro)
@@ -1,27 +1,6 @@
+<?xml version="1.0" ?>
 <robot xmlns:xacro="http://www.ros.org/wiki/xacro" name="valkyrie">
-	<xacro:property name="leg_mesh_dir" value="package://val_description/model/meshes/legs"/>
-    <xacro:property name="arm_mesh_dir" value="package://val_description/model/meshes/arms"/>
-    <xacro:property name="waist_mesh_dir" value="package://val_description/model/meshes/torso"/>
-    <xacro:property name="head_mesh_dir" value="package://val_description/model/meshes/head"/>
-    <xacro:property name="pelvis_mesh_dir" value="package://val_description/model/meshes/pelvis"/>
-    <xacro:property name="fingers_mesh_dir" value="package://val_description/model/meshes/fingers"/>
-    <xacro:property name="robot_type_suffix" value="_sim"/>
-    <xacro:include filename="../../model/robots/common/xacro/generic_models.xacro" />
-    <xacro:include filename="../../common/xacro/nodes/valkyrie_nodes.xacro"/>
-    <xacro:include filename="../../model/robots/common/xacro/sensors/sensor_transforms.xacro"/>
-    <xacro:include filename="../../model/robots/common/xacro/config/valkyrie_D_transmissions.xacro" />
-    <xacro:include filename="../../common/xacro/serial_numbers/valkyrie_D_serials.xacro"/>
-    <xacro:include filename="../../common/xacro/api/valkyrie_D_api.xacro"/>
-    <xacro:include filename="../../common/xacro/dev_ports/valkyrie_D_ports.xacro"/>
-    <!-- Pelvis include -->
-    <xacro:include filename="../../model/robots/common/xacro/pelvis/pelvis_includes.xacro"/>
-    <!-- Leg include -->
-    <xacro:include filename="../../model/robots/common/xacro/leg/leg_includes.xacro"/>
-    <!-- Head include -->
-    <xacro:include filename="../../model/robots/common/xacro/head/head_includes.xacro"/>
-    <!-- Arm include -->
-    <xacro:include filename="../../model/robots/common/xacro/arm/arm_includes.xacro"/>
-    <!-- Waist include -->
-    <xacro:include filename="../../model/robots/common/xacro/waist/waist_includes.xacro"/>
-    <xacro:include filename="../../model/robots/common/xacro/valkyrie_arm_mass_sims_base_hw.xacro"/>
+	<xacro:property name="robot_type_suffix" value="_sim"/>
+    <xacro:include filename="./valkyrie_generic.xacro"/>
+    <xacro:valkyrie_generic suffix="D"/>
 </robot>

File: model/robots/valkyrie_E.xacro (robot description, xacro)
@@ -1,28 +1,6 @@
-<robot xmlns:xacro="http://www.ros.org/wiki/xacro" name="ValkyrieE">
-	<xacro:property name="leg_mesh_dir" value="package://val_description/model/meshes/legs"/>
-    <xacro:property name="arm_mesh_dir" value="package://val_description/model/meshes/arms"/>
-    <xacro:property name="waist_mesh_dir" value="package://val_description/model/meshes/torso"/>
-    <xacro:property name="head_mesh_dir" value="package://val_description/model/meshes/head"/>
-    <xacro:property name="pelvis_mesh_dir" value="package://val_description/model/meshes/pelvis"/>
-    <xacro:property name="fingers_mesh_dir" value="package://val_description/model/meshes/fingers"/>
-    <xacro:property name="robot_type_suffix" value=""/>
-	<xacro:include filename="../../model/robots/common/xacro/generic_models.xacro" />
-    <xacro:include filename="../../common/xacro/nodes/valkyrie_nodes.xacro"/>
-    <xacro:include filename="../../model/robots/common/xacro/sensors/sensor_transforms.xacro"/>
-    <xacro:include filename="../../model/robots/common/xacro/config/valkyrie_E_transmissions.xacro" />
-	<xacro:include filename="../../common/xacro/serial_numbers/valkyrie_E_serials.xacro"/>
-    <xacro:include filename="../../common/xacro/api/valkyrie_E_api.xacro"/>
-    <xacro:include filename="../../common/xacro/dev_ports/valkyrie_E_ports.xacro"/>
-    <xacro:include filename="../../model/robots/common/xacro/common_bodies.xacro" />
-    <!-- Pelvis include -->
-    <xacro:include filename="../../model/robots/common/xacro/pelvis/pelvis_includes.xacro"/>
-    <!-- Leg include -->
-    <xacro:include filename="../../model/robots/common/xacro/leg/leg_includes.xacro"/>
-    <!-- Head include -->
-    <xacro:include filename="../../model/robots/common/xacro/head/head_includes.xacro"/>
-    <!-- Arm include -->
-    <xacro:include filename="../../model/robots/common/xacro/arm/arm_includes.xacro"/>
-    <!-- Waist include -->
-    <xacro:include filename="../../model/robots/common/xacro/waist/waist_includes.xacro"/>
-    <xacro:include filename="../../model/robots/common/xacro/valkyrie_base_hw.xacro"/>
+<?xml version="1.0" ?>
+<robot xmlns:xacro="http://www.ros.org/wiki/xacro" name="valkyrie">
+	<xacro:property name="robot_type_suffix" value=""/>
+    <xacro:include filename="./valkyrie_generic.xacro"/>
+    <xacro:valkyrie_generic suffix="E"/>
 </robot>

File: model/robots/valkyrie_E_arm_mass_sims.xacro (robot description, xacro)
@@ -1,27 +1,6 @@
+<?xml version="1.0" ?>
 <robot xmlns:xacro="http://www.ros.org/wiki/xacro" name="valkyrie">
-	<xacro:property name="leg_mesh_dir" value="package://val_description/model/meshes/legs"/>
-    <xacro:property name="arm_mesh_dir" value="package://val_description/model/meshes/arms"/>
-    <xacro:property name="waist_mesh_dir" value="package://val_description/model/meshes/torso"/>
-    <xacro:property name="head_mesh_dir" value="package://val_description/model/meshes/head"/>
-    <xacro:property name="pelvis_mesh_dir" value="package://val_description/model/meshes/pelvis"/>
-    <xacro:property name="fingers_mesh_dir" value="package://val_description/model/meshes/fingers"/>
-    <xacro:property name="robot_type_suffix" value="_sim"/>
-    <xacro:include filename="../../model/robots/common/xacro/generic_models.xacro" />
-    <xacro:include filename="../../common/xacro/nodes/valkyrie_nodes.xacro"/>
-    <xacro:include filename="../../model/robots/common/xacro/sensors/sensor_transforms.xacro"/>
-    <xacro:include filename="../../model/robots/common/xacro/config/valkyrie_E_transmissions.xacro" />
-    <xacro:include filename="../../common/xacro/serial_numbers/valkyrie_E_serials.xacro"/>
-    <xacro:include filename="../../common/xacro/api/valkyrie_E_api.xacro"/>
-    <xacro:include filename="../../common/xacro/dev_ports/valkyrie_E_ports.xacro"/>
-    <!-- Pelvis include -->
-    <xacro:include filename="../../model/robots/common/xacro/pelvis/pelvis_includes.xacro"/>
-    <!-- Leg include -->
-    <xacro:include filename="../../model/robots/common/xacro/leg/leg_includes.xacro"/>
-    <!-- Head include -->
-    <xacro:include filename="../../model/robots/common/xacro/head/head_includes.xacro"/>
-    <!-- Arm include -->
-    <xacro:include filename="../../model/robots/common/xacro/arm/arm_includes.xacro"/>
-    <!-- Waist include -->
-    <xacro:include filename="../../model/robots/common/xacro/waist/waist_includes.xacro"/>
-    <xacro:include filename="../../model/robots/common/xacro/valkyrie_arm_mass_sims_base_hw.xacro"/>
+	<xacro:property name="robot_type_suffix" value="_sim"/>
+    <xacro:include filename="./valkyrie_generic.xacro"/>
+    <xacro:valkyrie_generic suffix="E"/>
 </robot>
