Commit message: Changed prefixes for loading meshses

File: model/robots/valkyrie_sim.xacro (robot description, xacro)
@@ -6,10 +6,10 @@
     </gazebo>
     <schedule_topic_creator_file package="val_gazebo" relative_file_path="/configuration/valkyrie_sim_shm_topics.yaml"/>
-    <xacro:property name="leg_mesh_dir" value="model://val_description/model/meshes/legs"/>
-    <xacro:property name="arm_mesh_dir" value="model://val_description/model/meshes/arms"/>
-    <xacro:property name="waist_mesh_dir" value="model://val_description/model/meshes/torso"/>
-    <xacro:property name="head_mesh_dir" value="model://val_description/model/meshes/head"/>
-    <xacro:property name="pelvis_mesh_dir" value="model://val_description/model/meshes/pelvis"/>
-    <xacro:property name="fingers_mesh_dir" value="model://val_description/model/meshes/fingers"/>
+    <xacro:property name="leg_mesh_dir" value="package://val_description/model/meshes/legs"/>
+    <xacro:property name="arm_mesh_dir" value="package://val_description/model/meshes/arms"/>
+    <xacro:property name="waist_mesh_dir" value="package://val_description/model/meshes/torso"/>
+    <xacro:property name="head_mesh_dir" value="package://val_description/model/meshes/head"/>
+    <xacro:property name="pelvis_mesh_dir" value="package://val_description/model/meshes/pelvis"/>
+    <xacro:property name="fingers_mesh_dir" value="package://val_description/model/meshes/fingers"/>
     <xacro:property name="robot_type_suffix" value="_sim"/>
     <xacro:include filename="../../model/robots/common/xacro/generic_models.xacro" />

File: model/robots/valkyrie_sim_angled_legj1s.xacro (robot description, xacro)
@@ -6,10 +6,10 @@
     </gazebo>
     <schedule_topic_creator_file package="val_gazebo" relative_file_path="/configuration/valkyrie_sim_shm_topics.yaml"/>
-    <xacro:property name="leg_mesh_dir" value="model://val_description/model/meshes/legs_angled_j1s"/>
-    <xacro:property name="arm_mesh_dir" value="model://val_description/model/meshes/arms"/>
-    <xacro:property name="waist_mesh_dir" value="model://val_description/model/meshes/torso_angled_j1s"/>
-    <xacro:property name="head_mesh_dir" value="model://val_description/model/meshes/head"/>
-    <xacro:property name="pelvis_mesh_dir" value="model://val_description/model/meshes/pelvis_angled_j1s"/>
-    <xacro:property name="fingers_mesh_dir" value="model://val_description/model/meshes/fingers"/>
+    <xacro:property name="leg_mesh_dir" value="package://val_description/model/meshes/legs_angled_j1s"/>
+    <xacro:property name="arm_mesh_dir" value="package://val_description/model/meshes/arms"/>
+    <xacro:property name="waist_mesh_dir" value="package://val_description/model/meshes/torso_angled_j1s"/>
+    <xacro:property name="head_mesh_dir" value="package://val_description/model/meshes/head"/>
+    <xacro:property name="pelvis_mesh_dir" value="package://val_description/model/meshes/pelvis_angled_j1s"/>
+    <xacro:property name="fingers_mesh_dir" value="package://val_description/model/meshes/fingers"/>
     <xacro:property name="robot_type_suffix" value="_sim"/>
     <xacro:include filename="../../model/robots/common/xacro/generic_models.xacro" />

File: model/robots/valkyrie_sim_arm_mass_sims.xacro (robot description, xacro)
@@ -5,9 +5,9 @@
       </plugin>
     </gazebo>
-    <xacro:property name="leg_mesh_dir" value="model://val_description/model/meshes/legs"/>
-    <xacro:property name="arm_mesh_dir" value="model://val_description/model/meshes/arms"/>
-    <xacro:property name="waist_mesh_dir" value="model://val_description/model/meshes/torso"/>
-    <xacro:property name="head_mesh_dir" value="model://val_description/model/meshes/head"/>
-    <xacro:property name="pelvis_mesh_dir" value="model://val_description/model/meshes/pelvis"/>
+    <xacro:property name="leg_mesh_dir" value="package://val_description/model/meshes/legs"/>
+    <xacro:property name="arm_mesh_dir" value="package://val_description/model/meshes/arms"/>
+    <xacro:property name="waist_mesh_dir" value="package://val_description/model/meshes/torso"/>
+    <xacro:property name="head_mesh_dir" value="package://val_description/model/meshes/head"/>
+    <xacro:property name="pelvis_mesh_dir" value="package://val_description/model/meshes/pelvis"/>
     <xacro:property name="robot_type_suffix" value="_sim"/>
     <xacro:include filename="../../model/robots/common/xacro/generic_models.xacro" />

File: model/urdf/multisense_sl_remote.urdf (robot description, URDF)
Before this commit: robot multisense_sl, 11 links, 10 joints
Links:
- link multisense/hokuyo_link: geometry collision box size=0.08 0.06 0.04238; collision cylinder length=0.047 radius=0.024425

Commit message: Added fixed joint between the world and pelvis

File: model/robots/valkyrie_sim.xacro (robot description, xacro)
@@ -4,4 +4,9 @@
       </plugin>
     </gazebo>
+    <link name="world"/>
+    <joint name="fixed" type="fixed">
+        <parent link="world"/>
+        <child link="pelvis"/>
+    </joint>
     <xacro:property name="leg_mesh_dir" value="package://val_description/model/meshes/legs"/>
     <xacro:property name="arm_mesh_dir" value="package://val_description/model/meshes/arms"/>
