Commit message: Fixed an error where arm_mass_sims models were exactly the same full arm+hand models

File: model/robots/valkyrie_A.urdf.xacro (robot description, xacro)
@@ -2,4 +2,5 @@
 <robot xmlns:xacro="http://www.ros.org/wiki/xacro" name="ValkyrieA">
     <xacro:property name="robot_type_suffix" value=""/>
+    <xacro:property name="arm_mass_sims" default="false"/>
     <xacro:include filename="./valkyrie_generic.xacro"/>
     <xacro:valkyrie_generic suffix="A"/>

File: model/robots/valkyrie_A_arm_mass_sims.urdf.xacro (robot description, xacro)
@@ -2,4 +2,5 @@
 <robot xmlns:xacro="http://www.ros.org/wiki/xacro" name="valkyrie">
 	<xacro:property name="robot_type_suffix" value="_sim"/>
+	<xacro:property name="arm_mass_sims" default="true"/>
     <xacro:include filename="./valkyrie_generic.xacro"/>
     <xacro:valkyrie_generic suffix="A"/>

File: model/robots/valkyrie_B.urdf.xacro (robot description, xacro)
@@ -2,4 +2,5 @@
 <robot xmlns:xacro="http://www.ros.org/wiki/xacro" name="valkyrie">
 	<xacro:property name="robot_type_suffix" value=""/>
+	<xacro:property name="arm_mass_sims" default="false"/>
     <xacro:include filename="./valkyrie_generic.xacro"/>
     <xacro:valkyrie_generic suffix="B"/>

File: model/robots/valkyrie_B_arm_mass_sims.urdf.xacro (robot description, xacro)
@@ -2,4 +2,5 @@
 <robot xmlns:xacro="http://www.ros.org/wiki/xacro" name="valkyrie">
 	<xacro:property name="robot_type_suffix" value="_sim"/>
+	<xacro:property name="arm_mass_sims" default="true"/>
     <xacro:include filename="./valkyrie_generic.xacro"/>
     <xacro:valkyrie_generic suffix="B"/>

File: model/robots/valkyrie_C.urdf.xacro (robot description, xacro)
@@ -2,4 +2,5 @@
 <robot xmlns:xacro="http://www.ros.org/wiki/xacro" name="valkyrie">
 	<xacro:property name="robot_type_suffix" value=""/>
+	<xacro:property name="arm_mass_sims" default="false"/>
     <xacro:include filename="./valkyrie_generic.xacro"/>
     <xacro:valkyrie_generic suffix="C"/>

File: model/robots/valkyrie_C_arm_mass_sims.urdf.xacro (robot description, xacro)
@@ -2,4 +2,5 @@
 <robot xmlns:xacro="http://www.ros.org/wiki/xacro" name="valkyrie">
 	<xacro:property name="robot_type_suffix" value="_sim"/>
+	<xacro:property name="arm_mass_sims" default="true"/>
     <xacro:include filename="./valkyrie_generic.xacro"/>
     <xacro:valkyrie_generic suffix="C"/>

File: model/robots/valkyrie_D.urdf.xacro (robot description, xacro)
@@ -2,4 +2,5 @@
 <robot xmlns:xacro="http://www.ros.org/wiki/xacro" name="valkyrie">
 	<xacro:property name="robot_type_suffix" value=""/>
+	<xacro:property name="arm_mass_sims" default="false"/>
     <xacro:include filename="./valkyrie_generic.xacro"/>
     <xacro:valkyrie_generic suffix="D"/>

File: model/robots/valkyrie_D_arm_mass_sims.urdf.xacro (robot description, xacro)
@@ -2,4 +2,5 @@
 <robot xmlns:xacro="http://www.ros.org/wiki/xacro" name="valkyrie">
 	<xacro:property name="robot_type_suffix" value="_sim"/>
+	<xacro:property name="arm_mass_sims" default="true"/>
     <xacro:include filename="./valkyrie_generic.xacro"/>
     <xacro:valkyrie_generic suffix="D"/>

File: model/robots/valkyrie_E.urdf.xacro (robot description, xacro)
@@ -2,4 +2,5 @@
 <robot xmlns:xacro="http://www.ros.org/wiki/xacro" name="valkyrie">
 	<xacro:property name="robot_type_suffix" value=""/>
+	<xacro:property name="arm_mass_sims" default="false"/>
     <xacro:include filename="./valkyrie_generic.xacro"/>
     <xacro:valkyrie_generic suffix="E"/>

File: model/robots/valkyrie_E_arm_mass_sims.urdf.xacro (robot description, xacro)
@@ -2,4 +2,5 @@
 <robot xmlns:xacro="http://www.ros.org/wiki/xacro" name="valkyrie">
 	<xacro:property name="robot_type_suffix" value="_sim"/>
+	<xacro:property name="arm_mass_sims" default="true"/>
     <xacro:include filename="./valkyrie_generic.xacro"/>
     <xacro:valkyrie_generic suffix="E"/>

File: model/robots/valkyrie_generic.xacro (robot description, xacro)
@@ -17,5 +17,4 @@
         <xacro:include filename="${head}/common/xacro/api/valkyrie_${suffix}_api.xacro"/>
         <xacro:include filename="${head}/common/xacro/dev_ports/valkyrie_${suffix}_ports.xacro"/>
-        <xacro:include filename="${head}/model/robots/common/xacro/common_bodies.xacro" />
         <!-- Pelvis include -->
         <xacro:include filename="${head}/model/robots/common/xacro/pelvis/pelvis_includes.xacro"/>
@@ -28,12 +27,18 @@
         <!-- Waist include -->
         <xacro:include filename="${head}/model/robots/common/xacro/waist/waist_includes.xacro"/>
-        <xacro:property name="use_head" default="true"/>
-        <xacro:property name="use_right_arm" default="true"/>
-        <xacro:property name="use_right_hand" default="true"/>
-        <xacro:property name="use_right_leg" default="true"/>
-        <xacro:property name="use_left_arm" default="true"/>
-        <xacro:property name="use_left_hand" default="true"/>
-        <xacro:property name="use_left_leg" default="true"/>
-        <xacro:include filename="${head}/model/robots/common/xacro/valkyrie_base_hw.xacro"/>
+        <xacro:if value="${arm_mass_sims}">
+            <xacro:include filename="../../model/robots/common/xacro/valkyrie_arm_mass_sims_base_hw.xacro"/>
+        </xacro:if>
+        <xacro:unless value="${arm_mass_sims}">
+            <xacro:include filename="${head}/model/robots/common/xacro/common_bodies.xacro" />
+            <xacro:property name="use_head" default="true"/>
+            <xacro:property name="use_right_arm" default="true"/>
+            <xacro:property name="use_right_hand" default="true"/>
+            <xacro:property name="use_right_leg" default="true"/>
+            <xacro:property name="use_left_arm" default="true"/>
+            <xacro:property name="use_left_hand" default="true"/>
+            <xacro:property name="use_left_leg" default="true"/>
+            <xacro:include filename="${head}/model/robots/common/xacro/valkyrie_base_hw.xacro"/>
+        </xacro:unless>
     </xacro:macro>
 </robot>

Commit message: Adjusted parameters for ValkyrieA and generic

File: model/robots/valkyrie_A.urdf.xacro (robot description, xacro)
@@ -1,6 +1,7 @@
 <?xml version="1.0" ?>
 <robot xmlns:xacro="http://www.ros.org/wiki/xacro" name="ValkyrieA">
+    <xacro:arg name="arm_mass_sims" default="false"/>
     <xacro:property name="robot_type_suffix" value=""/>
-    <xacro:property name="arm_mass_sims" default="false"/>
+    <xacro:property name="arm_mass_sims" default="$(arg arm_mass_sims)"/>
     <xacro:include filename="./valkyrie_generic.xacro"/>
     <xacro:valkyrie_generic suffix="A"/>

File: model/robots/valkyrie_generic.xacro (robot description, xacro)
@@ -2,5 +2,5 @@
 <robot xmlns:xacro="http://www.ros.org/wiki/xacro" name="valkyrie">
     <xacro:macro name="valkyrie_generic" params="suffix">
-        <xacro:property name="head" default="../../"/>
+        <xacro:property name="head" default="$(find val_description)"/>
     	<xacro:property name="leg_mesh_dir" value="package://val_description/model/meshes/legs"/>
         <xacro:property name="arm_mesh_dir" value="package://val_description/model/meshes/arms"/>
@@ -27,16 +27,16 @@
         <!-- Waist include -->
         <xacro:include filename="${head}/model/robots/common/xacro/waist/waist_includes.xacro"/>
-        <xacro:if value="${arm_mass_sims}">
-            <xacro:include filename="../../model/robots/common/xacro/valkyrie_arm_mass_sims_base_hw.xacro"/>
+        <xacro:if value="$(arg arm_mass_sims)">
+            <xacro:include filename="${head}/model/robots/common/xacro/valkyrie_arm_mass_sims_base_hw.xacro"/>
         </xacro:if>
-        <xacro:unless value="${arm_mass_sims}">
+        <xacro:unless value="$(arg arm_mass_sims)">
             <xacro:include filename="${head}/model/robots/common/xacro/common_bodies.xacro" />
-            <xacro:property name="use_head" default="true"/>
-            <xacro:property name="use_right_arm" default="true"/>
-            <xacro:property name="use_right_hand" default="true"/>
-            <xacro:property name="use_right_leg" default="true"/>
-            <xacro:property name="use_left_arm" default="true"/>
-            <xacro:property name="use_left_hand" default="true"/>
-            <xacro:property name="use_left_leg" default="true"/>
+            <xacro:property name="use_head" default="$(arg use_head)"/>
+            <xacro:property name="use_right_arm" default="$(arg use_right_arm)"/>
+            <xacro:property name="use_right_hand" default="$(arg use_right_hand)"/>
+            <xacro:property name="use_right_leg" default="$(arg use_right_leg)"/>
+            <xacro:property name="use_left_arm" default="$(arg use_left_arm)"/>
+            <xacro:property name="use_left_hand" default="$(arg use_left_hand)"/>
+            <xacro:property name="use_left_leg" default="$(arg use_left_leg)"/>
             <xacro:include filename="${head}/model/robots/common/xacro/valkyrie_base_hw.xacro"/>
         </xacro:unless>
