Commit message: Support separate gains for sim versus hw

File: model/robots/common/xacro/arm/arm_includes.xacro (robot description, xacro)
@@ -6,5 +6,5 @@
 	<xacro:include filename="$(find val_description)/common/xacro/joint_names/valkyrie_joint_names.xacro"/>
 	<xacro:include filename="$(find val_description)/common/xacro/actuator_names/valkyrie_actuator_names.xacro"/>
-	<xacro:include filename="$(find val_description)/model/robots/common/xacro/gains.xacro"/>
+	<xacro:include filename="$(find val_description)/model/robots/common/xacro/gains${robot_type_suffix}.xacro"/>
 	<xacro:include filename="$(find val_description)/model/robots/common/xacro/gazebo_hand_contact.xacro"/>
 	<xacro:include filename="$(find val_description)/model/robots/common/xacro/arm/arm.xacro"/>

File: model/robots/common/xacro/gains_sim.xacro (robot description, xacro)
@@ -1,58 +1,6 @@
 <robot xmlns:xacro="http://www.ros.org/wiki/xacro" name="valkyrie_nodes">
-    <xacro:property name="ForearmYawKd" value="0.0" />
-    <xacro:property name="ForearmYawKi" value="0.0" />
-    <xacro:property name="WristPitchKp" value="500" />
-    <xacro:property name="WristPitchKd" value="0" />
-    <xacro:property name="WristPitchKi" value="0.0" />
-    <xacro:property name="WristRollKp" value="500" />
-    <xacro:property name="WristRollKd" value="0" />
-    <xacro:property name="WristRollKi" value="0.0" />
+    <!-- Get the hardware gains -->
+    <xacro:include filename="$(find val_description)/model/robots/common/xacro/gains.xacro"/>
+    <!-- Override only those properties that need to be different for sim -->
     <xacro:property name="LowerNeckPitchKp" value="150" />
-    <xacro:property name="LowerNeckPitchKd" value="3" />
-    <xacro:property name="LowerNeckPitchKi" value="3" />
-    <xacro:property name="NeckYawKp" value="150" />
-    <xacro:property name="NeckYawKd" value="3" />
-    <xacro:property name="NeckYawKi" value="0.0" />
-    <xacro:property name="UpperNeckPitchKp" value="150" />
-    <xacro:property name="UpperNeckPitchKd" value="3" />
-    <xacro:property name="UpperNeckPitchKi" value="0.0" />
-    <xacro:property name="ThumbRollKp" value="5.0" />
-    <xacro:property name="ThumbRollKd" value="0.0" />
-    <xacro:property name="ThumbRollKi" value="0.0" />
-    <xacro:property name="ThumbPitch1Kp" value="5.0" />
-    <xacro:property name="ThumbPitch1Kd" value="0.0" />
-    <xacro:property name="ThumbPitch1Ki" value="0.0" />
-    <xacro:property name="ThumbPitch2Kp" value="5.0" />
-    <xacro:property name="ThumbPitch2Kd" value="0.0" />
-    <xacro:property name="ThumbPitch2Ki" value="0.0" />
-    <xacro:property name="ThumbPitch3Kp" value="5.0" />
-    <xacro:property name="ThumbPitch3Kd" value="0.0" />
-    <xacro:property name="ThumbPitch3Ki" value="0.0" />
-    <xacro:property name="IndexFingerPitch1Kp" value="5.0" />
-    <xacro:property name="IndexFingerPitch1Kd" value="0.0" />
-    <xacro:property name="IndexFingerPitch1Ki" value="0.0" />
-    <xacro:property name="IndexFingerPitch2Kp" value="5.0" />
-    <xacro:property name="IndexFingerPitch2Kd" value="0.0" />
-    <xacro:property name="IndexFingerPitch2Ki" value="0.0" />
-    <xacro:property name="IndexFingerPitch3Kp" value="5.0" />
-    <xacro:property name="IndexFingerPitch3Kd" value="0.0" />
-    <xacro:property name="IndexFingerPitch3Ki" value="0.0" />
-    <xacro:property name="MiddleFingerPitch1Kp" value="5.0" />
-    <xacro:property name="MiddleFingerPitch1Kd" value="0.0" />
-    <xacro:property name="MiddleFingerPitch1Ki" value="0.0" />
-    <xacro:property name="MiddleFingerPitch2Kp" value="5.0" />
-    <xacro:property name="MiddleFingerPitch2Kd" value="0.0" />
-    <xacro:property name="MiddleFingerPitch2Ki" value="0.0" />
-    <xacro:property name="MiddleFingerPitch3Kp" value="5.0" />
-    <xacro:property name="MiddleFingerPitch3Kd" value="0.0" />
-    <xacro:property name="MiddleFingerPitch3Ki" value="0.0" />
-    <xacro:property name="PinkyPitch1Kp" value="5.0" />
-    <xacro:property name="PinkyPitch1Kd" value="0.0" />
-    <xacro:property name="PinkyPitch1Ki" value="0.0" />
-    <xacro:property name="PinkyPitch2Kp" value="5.0" />
-    <xacro:property name="PinkyPitch2Kd" value="0.0" />
-    <xacro:property name="PinkyPitch2Ki" value="0.0" />
-    <xacro:property name="PinkyPitch3Kp" value="5.0" />
-    <xacro:property name="PinkyPitch3Kd" value="0.0" />
-    <xacro:property name="PinkyPitch3Ki" value="0.0" />
 </robot>

File: model/robots/common/xacro/head/head_includes.xacro (robot description, xacro)
@@ -7,5 +7,5 @@
 	<xacro:include filename="$(find val_description)/common/xacro/joint_names/valkyrie_joint_names.xacro"/>
 	<xacro:include filename="$(find val_description)/common/xacro/actuator_names/valkyrie_actuator_names.xacro"/>
-	<xacro:include filename="$(find val_description)/model/robots/common/xacro/gains.xacro"/>
+	<xacro:include filename="$(find val_description)/model/robots/common/xacro/gains${robot_type_suffix}.xacro"/>
 	<xacro:include filename="$(find val_description)/model/robots/common/xacro/head/head.xacro"/>
 </robot>

File: model/robots/common/xacro/leg/angled_j1s_includes.xacro (robot description, xacro)
@@ -7,5 +7,5 @@
 	<xacro:include filename="$(find val_description)/common/xacro/joint_names/valkyrie_joint_names.xacro"/>
 	<xacro:include filename="$(find val_description)/common/xacro/actuator_names/valkyrie_actuator_names.xacro"/>
-	<xacro:include filename="$(find val_description)/model/robots/common/xacro/gains.xacro"/>
+	<xacro:include filename="$(find val_description)/model/robots/common/xacro/gains${robot_type_suffix}.xacro"/>
 	<xacro:include filename="$(find val_description)/model/robots/common/xacro/sensors/ati_force_torque.xacro"/>
 	<xacro:include filename="$(find val_description)/model/robots/common/xacro/leg/leg.xacro"/>

File: model/robots/common/xacro/leg/leg_includes.xacro (robot description, xacro)
@@ -6,5 +6,5 @@
 	<xacro:include filename="$(find val_description)/common/xacro/joint_names/valkyrie_joint_names.xacro"/>
 	<xacro:include filename="$(find val_description)/common/xacro/actuator_names/valkyrie_actuator_names.xacro"/>
-	<xacro:include filename="$(find val_description)/model/robots/common/xacro/gains.xacro"/>
+	<xacro:include filename="$(find val_description)/model/robots/common/xacro/gains${robot_type_suffix}.xacro"/>
 	<xacro:include filename="$(find val_description)/model/robots/common/xacro/sensors/ati_force_torque.xacro"/>
 	<xacro:include filename="$(find val_description)/model/robots/common/xacro/leg/leg.xacro"/>

File: model/robots/common/xacro/thumb/thumb.xacro (robot description, xacro)
@@ -7,5 +7,5 @@
   <xacro:include filename="$(find val_description)/model/robots/common/xacro/thumb/mass_parameters.xacro"/>
   <xacro:include filename="$(find val_description)/model/robots/common/xacro/thumb/mechanical_info.xacro"/>
-  <xacro:include filename="$(find val_description)/model/robots/common/xacro/gains.xacro"/>
+  <xacro:include filename="$(find val_description)/model/robots/common/xacro/gains${robot_type_suffix}.xacro"/>
   <xacro:include filename="$(find val_description)/model/robots/common/xacro/gazebo_hand_contact.xacro"/>
   <xacro:macro name="make_thumb" params="prefix reflect thumb_root_link">

File: model/robots/forearm_left.xacro (robot description, xacro)
@@ -2,4 +2,5 @@
     <xacro:property name="arm_mesh_dir" value="package://val_description/model/meshes/arms"/>
     <xacro:property name="fingers_mesh_dir" value="package://val_description/model/meshes/fingers"/>
+    <xacro:property name="robot_type_suffix" value=""/>
     <xacro:include filename="$(find val_description)/common/xacro/nodes/valkyrie_nodes.xacro"/>
     <xacro:include filename="$(find val_description)/model/robots/common/xacro/generic_models.xacro" />

File: model/robots/forearm_right.xacro (robot description, xacro)
@@ -2,4 +2,5 @@
     <xacro:property name="arm_mesh_dir" value="package://val_description/model/meshes/arms"/>
     <xacro:property name="fingers_mesh_dir" value="package://val_description/model/meshes/fingers"/>
+    <xacro:property name="robot_type_suffix" value=""/>
     <xacro:include filename="$(find val_description)/common/xacro/nodes/valkyrie_nodes.xacro"/>
     <xacro:include filename="$(find val_description)/model/robots/common/xacro/generic_models.xacro" />

File: model/robots/forearm_sim_right.xacro (robot description, xacro)
@@ -9,4 +9,5 @@
     <xacro:property name="arm_mesh_dir" value="package://val_description/model/meshes/arms"/>
     <xacro:property name="fingers_mesh_dir" value="package://val_description/model/meshes/fingers"/>
+    <xacro:property name="robot_type_suffix" value="_sim"/>
     <xacro:include filename="$(find val_description)/common/xacro/nodes/valkyrie_sim_nodes.xacro"/>
     <xacro:include filename="$(find val_description)/model/robots/common/xacro/generic_models.xacro" />

File: model/robots/imu_test.xacro (robot description, xacro)
@@ -1,8 +1,9 @@
 <robot xmlns:xacro="http://www.ros.org/wiki/xacro" name="valkyrie">
     <xacro:property name="mesh_root" value="package://val_description/model/meshes"/>
+    <xacro:property name="pelvis_mesh_dir" value="package://val_description/model/meshes/pelvis"/>
+    <xacro:property name="robot_type_suffix" value=""/>
     <xacro:include filename="$(find val_description)/common/xacro/nodes/valkyrie_nodes.xacro"/>
     <xacro:include filename="$(find val_description)/model/robots/common/xacro/generic_models.xacro" />
     <xacro:include filename="$(find val_description)/model/robots/common/xacro/common_bodies.xacro" />
-    <xacro:include filename="$(find val_description)/model/robots/common/xacro/valkyrie_imu_base.xacro"/>
     <xacro:include filename="$(find val_description)/common/xacro/serial_numbers/valkyrie_C_serials.xacro"/>
     <xacro:include filename="$(find val_description)/common/xacro/dev_ports/valkyrie_imu_test_ports.xacro"/>
@@ -10,4 +11,4 @@
     <xacro:include filename="$(find val_description)/model/robots/common/xacro/head/head_includes.xacro"/>
     <xacro:include filename="$(find val_description)/model/robots/common/xacro/sensors/sensor_transforms.xacro"/>
-    <xacro:property name="pelvis_mesh_dir" value="package://val_description/model/meshes/pelvis"/>
+    <xacro:include filename="$(find val_description)/model/robots/common/xacro/valkyrie_imu_base.xacro"/>
 </robot>

File: model/robots/leg_left.xacro (robot description, xacro)
@@ -2,4 +2,5 @@
     <link name="world"/>
     <xacro:property name="leg_mesh_dir" value="package://val_description/model/meshes/legs"/>
+    <xacro:property name="robot_type_suffix" value=""/>
     <xacro:property name="TorsoTransmissionType" value="robot_transmission_interface::TorsoPushrodTransmissionLoader"/>
     <xacro:property name="AnkleTransmissionType" value="robot_transmission_interface::AnklePushrodTransmissionLoader"/>

File: model/robots/leg_right.xacro (robot description, xacro)
@@ -2,4 +2,5 @@
     <link name="world"/>
     <xacro:property name="leg_mesh_dir" value="package://val_description/model/meshes/legs"/>
+    <xacro:property name="robot_type_suffix" value=""/>
     <xacro:property name="TorsoTransmissionType" value="robot_transmission_interface::TorsoPushrodTransmissionLoader"/>
     <xacro:property name="AnkleTransmissionType" value="robot_transmission_interface::AnklePushrodTransmissionLoader"/>

File: model/robots/valkyrie_A.xacro (robot description, xacro)
@@ -6,4 +6,5 @@
     <xacro:property name="pelvis_mesh_dir" value="package://val_description/model/meshes/pelvis"/>
     <xacro:property name="fingers_mesh_dir" value="package://val_description/model/meshes/fingers"/>
+    <xacro:property name="robot_type_suffix" value=""/>
 	<xacro:include filename="$(find val_description)/model/robots/common/xacro/generic_models.xacro" />
     <xacro:include filename="$(find val_description)/common/xacro/nodes/valkyrie_nodes.xacro"/>

File: model/robots/valkyrie_A_arm_mass_sims.xacro (robot description, xacro)
@@ -6,4 +6,5 @@
     <xacro:property name="pelvis_mesh_dir" value="package://val_description/model/meshes/pelvis"/>
     <xacro:property name="fingers_mesh_dir" value="package://val_description/model/meshes/fingers"/>
+    <xacro:property name="robot_type_suffix" value="_sim"/>
     <xacro:include filename="$(find val_description)/model/robots/common/xacro/generic_models.xacro" />
     <xacro:include filename="$(find val_description)/common/xacro/nodes/valkyrie_nodes.xacro"/>

File: model/robots/valkyrie_B.xacro (robot description, xacro)
@@ -6,4 +6,5 @@
     <xacro:property name="pelvis_mesh_dir" value="package://val_description/model/meshes/pelvis"/>
     <xacro:property name="fingers_mesh_dir" value="package://val_description/model/meshes/fingers"/>
+    <xacro:property name="robot_type_suffix" value=""/>
 	<xacro:include filename="$(find val_description)/model/robots/common/xacro/generic_models.xacro" />
     <xacro:include filename="$(find val_description)/common/xacro/nodes/valkyrie_nodes.xacro"/>

File: model/robots/valkyrie_B_arm_mass_sims.xacro (robot description, xacro)
@@ -6,4 +6,5 @@
     <xacro:property name="pelvis_mesh_dir" value="package://val_description/model/meshes/pelvis"/>
     <xacro:property name="fingers_mesh_dir" value="package://val_description/model/meshes/fingers"/>
+    <xacro:property name="robot_type_suffix" value="_sim"/>
     <xacro:include filename="$(find val_description)/model/robots/common/xacro/generic_models.xacro" />
     <xacro:include filename="$(find val_description)/common/xacro/nodes/valkyrie_nodes.xacro"/>

File: model/robots/valkyrie_C.xacro (robot description, xacro)
@@ -6,4 +6,5 @@
     <xacro:property name="pelvis_mesh_dir" value="package://val_description/model/meshes/pelvis"/>
     <xacro:property name="fingers_mesh_dir" value="package://val_description/model/meshes/fingers"/>
+    <xacro:property name="robot_type_suffix" value=""/>
 	<xacro:include filename="$(find val_description)/model/robots/common/xacro/generic_models.xacro" />
     <xacro:include filename="$(find val_description)/common/xacro/nodes/valkyrie_nodes.xacro"/>

File: model/robots/valkyrie_C_arm_mass_sims.xacro (robot description, xacro)
@@ -6,4 +6,5 @@
     <xacro:property name="pelvis_mesh_dir" value="package://val_description/model/meshes/pelvis"/>
     <xacro:property name="fingers_mesh_dir" value="package://val_description/model/meshes/fingers"/>
+    <xacro:property name="robot_type_suffix" value="_sim"/>
     <xacro:include filename="$(find val_description)/model/robots/common/xacro/generic_models.xacro" />
     <xacro:include filename="$(find val_description)/common/xacro/nodes/valkyrie_nodes.xacro"/>

File: model/robots/valkyrie_D.xacro (robot description, xacro)
@@ -6,4 +6,5 @@
     <xacro:property name="pelvis_mesh_dir" value="package://val_description/model/meshes/pelvis"/>
     <xacro:property name="fingers_mesh_dir" value="package://val_description/model/meshes/fingers"/>
+    <xacro:property name="robot_type_suffix" value=""/>
 	<xacro:include filename="$(find val_description)/model/robots/common/xacro/generic_models.xacro" />
     <xacro:include filename="$(find val_description)/common/xacro/nodes/valkyrie_nodes.xacro"/>

File: model/robots/valkyrie_D_arm_mass_sims.xacro (robot description, xacro)
@@ -6,4 +6,5 @@
     <xacro:property name="pelvis_mesh_dir" value="package://val_description/model/meshes/pelvis"/>
     <xacro:property name="fingers_mesh_dir" value="package://val_description/model/meshes/fingers"/>
+    <xacro:property name="robot_type_suffix" value="_sim"/>
     <xacro:include filename="$(find val_description)/model/robots/common/xacro/generic_models.xacro" />
     <xacro:include filename="$(find val_description)/common/xacro/nodes/valkyrie_nodes.xacro"/>
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