Commit message: Changed limit xacros to virtual wall limits

File: model/robots/common/xacro/arm/joint_limits.xacro (robot description, xacro)
@@ -8,15 +8,15 @@
   <xacro:property name="WristRollTorqueLimit" value="14" />
   <xacro:property name="WristPitchTorqueLimit" value="14" />
-  <xacro:property name="ShoulderPitchPositionLimit_Lower" value="-2.85" />
-  <xacro:property name="ShoulderRollPositionLimit_Lower" value="-1.519" />
-  <xacro:property name="ShoulderYawPositionLimit_Lower" value="-3.1" />
-  <xacro:property name="ElbowPitchPositionLimit_Lower" value="-2.174" />
+  <xacro:property name="ShoulderPitchPositionLimit_Lower" value="-2.78" />
+  <xacro:property name="ShoulderRollPositionLimit_Lower" value="-1.449" />
+  <xacro:property name="ShoulderYawPositionLimit_Lower" value="-3.03" />
+  <xacro:property name="ElbowPitchPositionLimit_Lower" value="-2.13" />
   <xacro:property name="ForearmYawPositionLimit_Lower" value="-2.019" />
   <xacro:property name="WristRollPositionLimit_Lower" value="-0.35" />
   <xacro:property name="WristPitchPositionLimit_Lower" value="-0.6" />
-  <xacro:property name="ShoulderPitchPositionLimit_Upper" value="2.0" />
-  <xacro:property name="ShoulderRollPositionLimit_Upper" value="1.266" />
-  <xacro:property name="ShoulderYawPositionLimit_Upper" value="2.18" />
-  <xacro:property name="ElbowPitchPositionLimit_Upper" value="0.12" />
+  <xacro:property name="ShoulderPitchPositionLimit_Upper" value="1.93" />
+  <xacro:property name="ShoulderRollPositionLimit_Upper" value="1.196" />
+  <xacro:property name="ShoulderYawPositionLimit_Upper" value="3.03" />
+  <xacro:property name="ElbowPitchPositionLimit_Upper" value="0.04" />
   <xacro:property name="ForearmYawPositionLimit_Upper" value="3.14" />
   <xacro:property name="WristRollPositionLimit_Upper" value="0.35" />

File: model/robots/common/xacro/leg/joint_limits.xacro (robot description, xacro)
@@ -7,14 +7,14 @@
   <xacro:property name="AnklePitchTorqueLimit" value="205" />
   <xacro:property name="AnkleRollTorqueLimit" value="205" />
-  <xacro:property name="HipYawPositionLimit_Lower" value="-1.1" />
-  <xacro:property name="HipRollPositionLimit_Lower" value="-0.5515" />
-  <xacro:property name="HipPitchPositionLimit_Lower" value="-2.42" />
-  <xacro:property name="KneePitchPositionLimit_Lower" value="-0.083" />
+  <xacro:property name="HipYawPositionLimit_Lower" value="-1.03" />
+  <xacro:property name="HipRollPositionLimit_Lower" value="-0.4815" />
+  <xacro:property name="HipPitchPositionLimit_Lower" value="-1.63" />
+  <xacro:property name="KneePitchPositionLimit_Lower" value="-0.055" />
   <xacro:property name="AnklePitchPositionLimit_Lower" value="-0.93" />
   <xacro:property name="AnkleRollPositionLimit_Lower" value="-0.4" />
-  <xacro:property name="HipYawPositionLimit_Upper" value="0.4141" />
-  <xacro:property name="HipRollPositionLimit_Upper" value="0.467" />
-  <xacro:property name="HipPitchPositionLimit_Upper" value="1.619" />
-  <xacro:property name="KneePitchPositionLimit_Upper" value="2.057" />
+  <xacro:property name="HipYawPositionLimit_Upper" value="0.38" />
+  <xacro:property name="HipRollPositionLimit_Upper" value="0.45" />
+  <xacro:property name="HipPitchPositionLimit_Upper" value="1.549" />
+  <xacro:property name="KneePitchPositionLimit_Upper" value="1.95" />
   <xacro:property name="AnklePitchPositionLimit_Upper" value="0.65" />
   <xacro:property name="AnkleRollPositionLimit_Upper" value="0.4" />

File: model/robots/common/xacro/waist/joint_limits.xacro (robot description, xacro)
@@ -4,8 +4,8 @@
   <xacro:property name="TorsoPitchTorqueLimit" value="150" />
   <xacro:property name="TorsoRollTorqueLimit" value="150" />
-  <xacro:property name="TorsoYawPositionLimit_Lower" value="-1.329" />
+  <xacro:property name="TorsoYawPositionLimit_Lower" value="-1.259" />
   <xacro:property name="TorsoPitchPositionLimit_Lower" value="-0.13" />
   <xacro:property name="TorsoRollPositionLimit_Lower" value="-0.23" />
-  <xacro:property name="TorsoYawPositionLimit_Upper" value="1.181" />
+  <xacro:property name="TorsoYawPositionLimit_Upper" value="1.111" />
   <xacro:property name="TorsoPitchPositionLimit_Upper" value="0.666" />
   <xacro:property name="TorsoRollPositionLimit_Upper" value="0.255" />
