Commit message: committing local changes

File: common/xacro/serial_numbers/forearm_left_testbench_serials.xacro (robot description, xacro)
@@ -1,4 +1,4 @@
 <robot xmlns:xacro="http://www.ros.org/wiki/xacro" name="forearm_testbench">
-	<xacro:property name="forearm_serial_number" value="v_h_005" />
-	<xacro:property name="forearm_yaw_serial_number" value="v_g_016" />
+	<xacro:property name="forearm_serial_number" value="v_h_007" />
+	<xacro:property name="forearm_yaw_serial_number" value="v_g_018" />
 </robot>

File: common/xacro/serial_numbers/forearm_testbench_serials.xacro (robot description, xacro)
@@ -1,4 +1,4 @@
 <robot xmlns:xacro="http://www.ros.org/wiki/xacro" name="forearm_testbench">
-	<xacro:property name="forearm_yaw_serial_number" value="v_g_017" />
-	<xacro:property name="hand_serial_number" value="v_h_008" />
+	<xacro:property name="forearm_yaw_serial_number" value="v_g_018" />
+	<xacro:property name="hand_serial_number" value="v_h_007" />
 </robot>
