Commit message: Capture demo config

File: common/xacro/serial_numbers/valkyrie_A_serials.xacro (robot description, xacro)
@@ -16,6 +16,6 @@
 	<xacro:property name="leftArmJ3SerialNumber" value="v_f_005" />
 	<xacro:property name="leftArmJ4SerialNumber" value="v_f_020" />
-        <xacro:property name="leftArmJ5SerialNumber" value="v_g_018" />
-        <xacro:property name="leftForearmSerialNumber" value="v_h_007"/>
+        <xacro:property name="leftArmJ5SerialNumber" value="v_g_016" />
+        <xacro:property name="leftForearmSerialNumber" value="v_h_005"/>
 	<xacro:property name="rightArmJ1SerialNumber" value="v_a_001" />
 	<xacro:property name="rightArmJ2SerialNumber" value="v_b_003" />

Commit message: adding uncommitted changes on console.  serials and thumb prox and pinky

File: common/xacro/serial_numbers/valkyrie_A_serials.xacro (robot description, xacro)
@@ -16,6 +16,6 @@
 	<xacro:property name="leftArmJ3SerialNumber" value="v_f_005" />
 	<xacro:property name="leftArmJ4SerialNumber" value="v_f_020" />
-        <xacro:property name="leftArmJ5SerialNumber" value="v_g_016" />
-        <xacro:property name="leftForearmSerialNumber" value="v_h_005"/>
+        <xacro:property name="leftArmJ5SerialNumber" value="v_g_018" />
+        <xacro:property name="leftForearmSerialNumber" value="v_h_007"/>
 	<xacro:property name="rightArmJ1SerialNumber" value="v_a_001" />
 	<xacro:property name="rightArmJ2SerialNumber" value="v_b_003" />

Commit message: Recalibrated index, middle, thumb prox and distal to fix slumpy fingers.

File: common/xacro/serial_numbers/valkyrie_A_serials.xacro (robot description, xacro)
@@ -22,6 +22,6 @@
 	<xacro:property name="rightArmJ3SerialNumber" value="v_f_004" />
 	<xacro:property name="rightArmJ4SerialNumber" value="v_f_003" />
-        <xacro:property name="rightArmJ5SerialNumber" value="v_g_017" />
-        <xacro:property name="rightForearmSerialNumber" value="v_h_008" />
+        <xacro:property name="rightArmJ5SerialNumber" value="v_g_012" />
+        <xacro:property name="rightForearmSerialNumber" value="v_h_006" />
 	<xacro:property name="neckJ1SerialNumber" value="v_g_006" />
 	<xacro:property name="neckJ2SerialNumber" value="v_g_007" />

Commit message: updated coeffs

File: common/xacro/serial_numbers/valkyrie_A_serials.xacro (robot description, xacro)
@@ -22,6 +22,6 @@
 	<xacro:property name="rightArmJ3SerialNumber" value="v_f_004" />
 	<xacro:property name="rightArmJ4SerialNumber" value="v_f_003" />
-        <xacro:property name="rightArmJ5SerialNumber" value="v_g_012" />
-        <xacro:property name="rightForearmSerialNumber" value="v_h_006" />
+        <xacro:property name="rightArmJ5SerialNumber" value="v_g_017" />
+        <xacro:property name="rightForearmSerialNumber" value="v_h_008" />
 	<xacro:property name="neckJ1SerialNumber" value="v_g_006" />
 	<xacro:property name="neckJ2SerialNumber" value="v_g_007" />
