Commit message: Coeffs and serial post-calibration

File: common/xacro/serial_numbers/valkyrie_B_serials.xacro (robot description, xacro)
@@ -18,5 +18,5 @@
         <xacro:property name="leftArmJ5SerialNumber" value="v_g_016" />
         <xacro:property name="leftForearmSerialNumber" value="v_h_005"/>
-	<xacro:property name="rightArmJ1SerialNumber" value="v_a_010" />
+	<xacro:property name="rightArmJ1SerialNumber" value="v_a_021" />
 	<xacro:property name="rightArmJ2SerialNumber" value="v_b_008" />
 	<xacro:property name="rightArmJ3SerialNumber" value="v_f_009" />
