Commit message: Changed val e serials

File: common/xacro/serial_numbers/valkyrie_E_serials.xacro (robot description, xacro)
@@ -12,5 +12,5 @@
         <xacro:property name="rightAnkleLeftActuatorSerialNumber" value="v_e_021" />
         <xacro:property name="rightAnkleRightActuatorSerialNumber" value="v_e_022" />
-	<xacro:property name="leftArmJ1SerialNumber" value="v_a_005" />
+	<xacro:property name="leftArmJ1SerialNumber" value="v_a_022" />
 	<xacro:property name="leftArmJ2SerialNumber" value="v_b_004" />
 	<xacro:property name="leftArmJ3SerialNumber" value="v_f_005" />
@@ -18,5 +18,5 @@
         <xacro:property name="leftArmJ5SerialNumber" value="v_g_018" />
         <xacro:property name="leftForearmSerialNumber" value="v_h_007"/>
-	<xacro:property name="rightArmJ1SerialNumber" value="v_a_001" />
+	<xacro:property name="rightArmJ1SerialNumber" value="v_a_010" />
 	<xacro:property name="rightArmJ2SerialNumber" value="v_b_003" />
 	<xacro:property name="rightArmJ3SerialNumber" value="v_f_004" />
@@ -28,6 +28,6 @@
 	<xacro:property name="neckJ3SerialNumber" value="v_g_008" />
 	<xacro:property name="trunkSerialNumber" value="v_a_004" />
-	<xacro:property name="waistRightActuatorSerialNumber" value="v_e_005" />
-	<xacro:property name="waistLeftActuatorSerialNumber" value="v_e_006" />
+	<xacro:property name="waistRightActuatorSerialNumber" value="v_e_025" />
+	<xacro:property name="waistLeftActuatorSerialNumber" value="v_e_026" />
 	<xacro:property name="left_foot_ATI_serial" value="FT17218" />
 	<xacro:property name="right_foot_ATI_serial" value="FT14018" />

Commit message: Final coeffs for trunk E

File: common/xacro/serial_numbers/valkyrie_E_serials.xacro (robot description, xacro)
@@ -28,6 +28,6 @@
 	<xacro:property name="neckJ3SerialNumber" value="v_g_008" />
 	<xacro:property name="trunkSerialNumber" value="v_a_004" />
-	<xacro:property name="waistRightActuatorSerialNumber" value="v_e_025" />
-	<xacro:property name="waistLeftActuatorSerialNumber" value="v_e_026" />
+	<xacro:property name="waistRightActuatorSerialNumber" value="v_e_026" />
+	<xacro:property name="waistLeftActuatorSerialNumber" value="v_e_025" />
 	<xacro:property name="left_foot_ATI_serial" value="FT17218" />
 	<xacro:property name="right_foot_ATI_serial" value="FT14018" />

Commit message: Zeroed (not calibrated) with jigs

File: common/xacro/serial_numbers/valkyrie_E_serials.xacro (robot description, xacro)
@@ -1,35 +1,35 @@
 <robot xmlns:xacro="http://www.ros.org/wiki/xacro" name="valkyrie_E_serials">
-	<xacro:property name="leftLegJ1SerialNumber" value="v_a_006" />
-        <xacro:property name="leftLegJ2SerialNumber" value="v_b_016" />
-    <xacro:property name="leftLegJ3SerialNumber" value="v_c_008" />
-    <xacro:property name="leftLegJ4SerialNumber" value="v_d_008" />
-    <xacro:property name="leftAnkleLeftActuatorSerialNumber" value="v_e_016" />
-        <xacro:property name="leftAnkleRightActuatorSerialNumber" value="v_e_015" />
-	<xacro:property name="rightLegJ1SerialNumber" value="v_a_003" />
-       <xacro:property name="rightLegJ2SerialNumber" value="v_b_017" />
-        <xacro:property name="rightLegJ3SerialNumber" value="v_c_009" />
-        <xacro:property name="rightLegJ4SerialNumber" value="v_d_009" />
-        <xacro:property name="rightAnkleLeftActuatorSerialNumber" value="v_e_021" />
-        <xacro:property name="rightAnkleRightActuatorSerialNumber" value="v_e_022" />
+	<xacro:property name="leftLegJ1SerialNumber" value="v_a_025" />
+        <xacro:property name="leftLegJ2SerialNumber" value="v_b_018" />
+    <xacro:property name="leftLegJ3SerialNumber" value="v_c_010" />
+    <xacro:property name="leftLegJ4SerialNumber" value="v_d_001" />
+    <xacro:property name="leftAnkleLeftActuatorSerialNumber" value="v_e_027" />
+        <xacro:property name="leftAnkleRightActuatorSerialNumber" value="v_e_028" />
+	<xacro:property name="rightLegJ1SerialNumber" value="v_a_023" />
+       <xacro:property name="rightLegJ2SerialNumber" value="v_b_020" />
+        <xacro:property name="rightLegJ3SerialNumber" value="v_c_011" />
+        <xacro:property name="rightLegJ4SerialNumber" value="v_d_010" />
+        <xacro:property name="rightAnkleLeftActuatorSerialNumber" value="v_e_029" />
+        <xacro:property name="rightAnkleRightActuatorSerialNumber" value="v_e_030" />
 	<xacro:property name="leftArmJ1SerialNumber" value="v_a_022" />
-	<xacro:property name="leftArmJ2SerialNumber" value="v_b_004" />
-	<xacro:property name="leftArmJ3SerialNumber" value="v_f_005" />
-	<xacro:property name="leftArmJ4SerialNumber" value="v_f_020" />
+	<xacro:property name="leftArmJ2SerialNumber" value="v_b_019" />
+	<xacro:property name="leftArmJ3SerialNumber" value="v_f_022" />
+	<xacro:property name="leftArmJ4SerialNumber" value="v_f_021" />
         <xacro:property name="leftArmJ5SerialNumber" value="v_g_018" />
         <xacro:property name="leftForearmSerialNumber" value="v_h_007"/>
 	<xacro:property name="rightArmJ1SerialNumber" value="v_a_010" />
-	<xacro:property name="rightArmJ2SerialNumber" value="v_b_003" />
-	<xacro:property name="rightArmJ3SerialNumber" value="v_f_004" />
-	<xacro:property name="rightArmJ4SerialNumber" value="v_f_003" />
+	<xacro:property name="rightArmJ2SerialNumber" value="v_b_015" />
+	<xacro:property name="rightArmJ3SerialNumber" value="v_f_023" />
+	<xacro:property name="rightArmJ4SerialNumber" value="v_f_002" />
         <xacro:property name="rightArmJ5SerialNumber" value="v_g_017" />
         <xacro:property name="rightForearmSerialNumber" value="v_h_008" />
-	<xacro:property name="neckJ1SerialNumber" value="v_g_006" />
-	<xacro:property name="neckJ2SerialNumber" value="v_g_007" />
-	<xacro:property name="neckJ3SerialNumber" value="v_g_008" />
-	<xacro:property name="trunkSerialNumber" value="v_a_004" />
+	<xacro:property name="neckJ1SerialNumber" value="v_g_022" />
+	<xacro:property name="neckJ2SerialNumber" value="v_g_021" />
+	<xacro:property name="neckJ3SerialNumber" value="v_g_023" />
+	<xacro:property name="trunkSerialNumber" value="v_a_024" />
 	<xacro:property name="waistRightActuatorSerialNumber" value="v_e_026" />
 	<xacro:property name="waistLeftActuatorSerialNumber" value="v_e_025" />
-	<xacro:property name="left_foot_ATI_serial" value="FT17218" />
-	<xacro:property name="right_foot_ATI_serial" value="FT14018" />
+	<xacro:property name="left_foot_ATI_serial" value="FT26293" />
+	<xacro:property name="right_foot_ATI_serial" value="FT26291" />
 	<xacro:property name="sim_ATI_serial" value="FT001SIM" />
 </robot>

Commit message: Update futek serial numbers after replacing load cells

File: common/xacro/serial_numbers/valkyrie_E_serials.xacro (robot description, xacro)
@@ -30,6 +30,6 @@
 	<xacro:property name="waistRightActuatorSerialNumber" value="v_e_026" />
 	<xacro:property name="waistLeftActuatorSerialNumber" value="v_e_025" />
-	<xacro:property name="left_foot_ATI_serial" value="FT26293" />
-	<xacro:property name="right_foot_ATI_serial" value="FT26291" />
+	<xacro:property name="left_foot_ATI_serial" value="FT27874" />
+	<xacro:property name="right_foot_ATI_serial" value="FT17216" />
 	<xacro:property name="sim_ATI_serial" value="FT001SIM" />
 </robot>

Commit message: Capture current Val E coeffs

File: common/xacro/serial_numbers/valkyrie_E_serials.xacro (robot description, xacro)
@@ -16,6 +16,6 @@
 	<xacro:property name="leftArmJ3SerialNumber" value="v_f_022" />
 	<xacro:property name="leftArmJ4SerialNumber" value="v_f_021" />
-        <xacro:property name="leftArmJ5SerialNumber" value="v_g_018" />
-        <xacro:property name="leftForearmSerialNumber" value="v_h_007"/>
+        <xacro:property name="leftArmJ5SerialNumber" value="v_g_016" />
+        <xacro:property name="leftForearmSerialNumber" value="v_h_005"/>
 	<xacro:property name="rightArmJ1SerialNumber" value="v_a_010" />
 	<xacro:property name="rightArmJ2SerialNumber" value="v_b_015" />

Commit message: Latest running Val E coeffs

File: common/xacro/serial_numbers/valkyrie_E_serials.xacro (robot description, xacro)
@@ -31,5 +31,5 @@
 	<xacro:property name="waistLeftActuatorSerialNumber" value="v_e_025" />
 	<xacro:property name="left_foot_ATI_serial" value="FT27874" />
-	<xacro:property name="right_foot_ATI_serial" value="FT17216" />
+	<xacro:property name="right_foot_ATI_serial" value="FT26293" />
 	<xacro:property name="sim_ATI_serial" value="FT001SIM" />
 </robot>

Commit message: update val E forearm serials and right shoulder pitch parameters.

File: common/xacro/serial_numbers/valkyrie_E_serials.xacro (robot description, xacro)
@@ -22,6 +22,6 @@
 	<xacro:property name="rightArmJ3SerialNumber" value="v_f_023" />
 	<xacro:property name="rightArmJ4SerialNumber" value="v_f_002" />
-        <xacro:property name="rightArmJ5SerialNumber" value="v_g_017" />
-        <xacro:property name="rightForearmSerialNumber" value="v_h_008" />
+        <xacro:property name="rightArmJ5SerialNumber" value="v_g_012" />
+        <xacro:property name="rightForearmSerialNumber" value="v_h_006" />
 	<xacro:property name="neckJ1SerialNumber" value="v_g_022" />
 	<xacro:property name="neckJ2SerialNumber" value="v_g_021" />

Commit message: Using unit C neck

File: common/xacro/serial_numbers/valkyrie_E_serials.xacro (robot description, xacro)
@@ -24,7 +24,7 @@
         <xacro:property name="rightArmJ5SerialNumber" value="v_g_012" />
         <xacro:property name="rightForearmSerialNumber" value="v_h_006" />
-	<xacro:property name="neckJ1SerialNumber" value="v_g_022" />
-	<xacro:property name="neckJ2SerialNumber" value="v_g_021" />
-	<xacro:property name="neckJ3SerialNumber" value="v_g_023" />
+	<xacro:property name="neckJ1SerialNumber" value="v_g_001" />
+	<xacro:property name="neckJ2SerialNumber" value="v_g_002" />
+	<xacro:property name="neckJ3SerialNumber" value="v_g_004" />
 	<xacro:property name="trunkSerialNumber" value="v_a_024" />
 	<xacro:property name="waistRightActuatorSerialNumber" value="v_e_026" />

Commit message: Updating coeffs from testing on the robot

File: common/xacro/serial_numbers/valkyrie_E_serials.xacro (robot description, xacro)
@@ -22,6 +22,6 @@
 	<xacro:property name="rightArmJ3SerialNumber" value="v_f_023" />
 	<xacro:property name="rightArmJ4SerialNumber" value="v_f_002" />
-        <xacro:property name="rightArmJ5SerialNumber" value="v_g_012" />
-        <xacro:property name="rightForearmSerialNumber" value="v_h_006" />
+        <xacro:property name="rightArmJ5SerialNumber" value="v_g_025" />
+        <xacro:property name="rightForearmSerialNumber" value="v_h_009" />
 	<xacro:property name="neckJ1SerialNumber" value="v_g_001" />
 	<xacro:property name="neckJ2SerialNumber" value="v_g_002" />
