Commit message: Improve fidelity of finger orientation relative to hand

File: model/robots/common/xacro/index_finger/frame_parameters.xacro (robot description, xacro)
@@ -3,5 +3,5 @@
   <xacro:property name="IndexFingerPitch1FrameOrigin_X" value="0.0022"/>
   <xacro:property name="IndexFingerPitch1FrameOrigin_Y" value="0.0976"/>
-  <xacro:property name="IndexFingerPitch1FrameOrigin_Z" value="0.0235"/>
+  <xacro:property name="IndexFingerPitch1FrameOrigin_Z" value="0.017"/>
   <xacro:property name="IndexFingerPitch1FrameOrientation_Roll" value="0.1745"/>
   <xacro:property name="IndexFingerPitch1FrameOrientation_Pitch" value="0.0"/>

File: model/robots/common/xacro/index_finger/index_finger.xacro (robot description, xacro)
@@ -38,6 +38,6 @@
     <xacro:revolute_joint_ex jointName="${prefix}${IndexFingerPitch1JointName}"
                           parent="${index_finger_root_link}" child="${prefix}IndexFingerPitch1Link"
-                          origin_xyz="${IndexFingerPitch1FrameOrigin_X} ${reflect * 0.0976} ${IndexFingerPitch1FrameOrigin_Z}"
-                          origin_rpy="${reflect * 0.1745} ${IndexFingerPitch1FrameOrientation_Pitch} ${IndexFingerPitch1FrameOrientation_Yaw}"
+                          origin_xyz="${IndexFingerPitch1FrameOrigin_X} ${reflect * IndexFingerPitch1FrameOrigin_Y} ${IndexFingerPitch1FrameOrigin_Z}"
+                          origin_rpy="${reflect * -0.02} ${IndexFingerPitch1FrameOrientation_Pitch} ${IndexFingerPitch1FrameOrientation_Yaw}"
                           axis="${IndexFingerPitch1RotationAxis}" damping="0.5" friction="0.5">
         <xacro:if value="${(reflect+1)/2}">

File: model/robots/common/xacro/pinky_finger/pinky_finger.xacro (robot description, xacro)
@@ -39,5 +39,5 @@
                           parent="${pinky_finger_root_link}" child="${prefix}PinkyPitch1Link"
                           origin_xyz="${PinkyPitch1FrameOrigin_X} ${reflect * 0.0838} ${PinkyPitch1FrameOrigin_Z}"
-                          origin_rpy="${reflect * -0.1222} ${PinkyPitch1FrameOrientation_Pitch} ${PinkyPitch1FrameOrientation_Yaw}"
+                          origin_rpy="${reflect * -0.22} ${PinkyPitch1FrameOrientation_Pitch} ${PinkyPitch1FrameOrientation_Yaw}"
                           axis="${PinkyFingerPitch1RotationAxis}" damping="0.5" friction="0.5">
         <xacro:if value="${(reflect+1)/2}">
