Commit message: Changes for focal
- Convert $(find val_description) references to relative paths, because find will look in an
installed location rather than in source.
- Work around a bug in xacro that is sometimes causing global properties to be unresolved
inside macros.

File: instance/instances/robots/actuator_testbench.xacro (robot description, xacro)
@@ -1,5 +1,5 @@
 <robot xmlns:xacro="http://www.ros.org/wiki/xacro" name="actuator_testbench">
 	<xacro:property name="instance" value="actuator_testbench" />
-	<xacro:include filename="$(find val_description)/common/xacro/serial_numbers/test_bench_serials.xacro" />
-    <xacro:include filename="$(find val_description)/instance/instances/robots/xacro/common/test_bench_template.xacro"/>
+	<xacro:include filename="../../../common/xacro/serial_numbers/test_bench_serials.xacro" />
+    <xacro:include filename="../../../instance/instances/robots/xacro/common/test_bench_template.xacro"/>
 </robot>

File: instance/instances/robots/forearm_testbench_left.xacro (robot description, xacro)
@@ -2,11 +2,11 @@
 	<xacro:property name="instance" value="forearm_testbench_left" />
 	<xacro:property name="prefix" value="left" />
-        <xacro:include filename="$(find val_description)/instance/instances/robots/xacro/firmware/firmware.xacro" />
-        <xacro:include filename="$(find val_description)/instance/instances/robots/xacro/firmware/forearm_firmware.xacro" />
-	<xacro:include filename="$(find val_description)/common/xacro/nodes/forearm_testbench_nodes_left.xacro" />
-	<xacro:include filename="$(find val_description)/common/xacro/serial_numbers/forearm_testbench_serials.xacro" />
-    <xacro:include filename="$(find val_description)/instance/instances/robots/xacro/mechanisms/mechanisms.xacro"/>
-    <xacro:include filename="$(find val_description)/common/xacro/joint_names/valkyrie_joint_names.xacro"/>
-    <xacro:include filename="$(find val_description)/common/xacro/firmware/valkyrie_firmware.xacro"/>
+    <xacro:include filename="../../../common/xacro/firmware/valkyrie_firmware.xacro"/>
+        <xacro:include filename="../../../instance/instances/robots/xacro/firmware/firmware.xacro" />
+        <xacro:include filename="../../../instance/instances/robots/xacro/firmware/forearm_firmware.xacro" />
+	<xacro:include filename="../../../common/xacro/nodes/forearm_testbench_nodes_left.xacro" />
+	<xacro:include filename="../../../common/xacro/serial_numbers/forearm_testbench_serials.xacro" />
+    <xacro:include filename="../../../instance/instances/robots/xacro/mechanisms/mechanisms.xacro"/>
+    <xacro:include filename="../../../common/xacro/joint_names/valkyrie_joint_names.xacro"/>
     <Channels>
     </Channels>

File: instance/instances/robots/forearm_testbench_right.xacro (robot description, xacro)
@@ -2,12 +2,12 @@
     <xacro:property name="instance" value="forearm_testbench_right" />
     <xacro:property name="prefix" value="right" />
-    <xacro:include filename="$(find val_description)/instance/instances/robots/xacro/firmware/firmware.xacro" />
-    <xacro:include filename="$(find val_description)/instance/instances/robots/xacro/firmware/forearm_firmware.xacro" />
-    <xacro:include filename="$(find val_description)/common/xacro/nodes/forearm_testbench_nodes.xacro" />
-    <xacro:include filename="$(find val_description)/common/xacro/serial_numbers/forearm_testbench_serials.xacro" />
-    <xacro:include filename="$(find val_description)/instance/instances/robots/xacro/mechanisms/mechanisms.xacro"/>
-    <xacro:include filename="$(find val_description)/instance/instances/robots/xacro/common/joint_calibration_angles.xacro"/>
-    <xacro:include filename="$(find val_description)/common/xacro/joint_names/valkyrie_joint_names.xacro"/>
-    <xacro:include filename="$(find val_description)/common/xacro/firmware/valkyrie_firmware.xacro"/>
+    <xacro:include filename="../../../instance/instances/robots/xacro/firmware/firmware.xacro" />
+    <xacro:include filename="../../../instance/instances/robots/xacro/firmware/forearm_firmware.xacro" />
+    <xacro:include filename="../../../common/xacro/nodes/forearm_testbench_nodes.xacro" />
+    <xacro:include filename="../../../common/xacro/serial_numbers/forearm_testbench_serials.xacro" />
+    <xacro:include filename="../../../instance/instances/robots/xacro/mechanisms/mechanisms.xacro"/>
+    <xacro:include filename="../../../instance/instances/robots/xacro/common/joint_calibration_angles.xacro"/>
+    <xacro:include filename="../../../common/xacro/joint_names/valkyrie_joint_names.xacro"/>
+    <xacro:include filename="../../../common/xacro/firmware/valkyrie_firmware.xacro"/>
     <Channels>
     </Channels>

File: instance/instances/robots/valkyrie_A.xacro (robot description, xacro)
@@ -1,5 +1,5 @@
 <robot xmlns:xacro="http://www.ros.org/wiki/xacro" name="valkyrie_A">
 	<xacro:property name="instance" value="valkyrie_A" />
-	<xacro:include filename="$(find val_description)/common/xacro/serial_numbers/valkyrie_A_serials.xacro" />
-    <xacro:include filename="$(find val_description)/instance/instances/robots/xacro/common/valkyrie_full_template.xacro"/>
+	<xacro:include filename="../../../common/xacro/serial_numbers/valkyrie_A_serials.xacro" />
+    <xacro:include filename="../../../instance/instances/robots/xacro/common/valkyrie_full_template.xacro"/>
 </robot>

File: instance/instances/robots/valkyrie_B.xacro (robot description, xacro)
@@ -1,5 +1,5 @@
 <robot xmlns:xacro="http://www.ros.org/wiki/xacro" name="valkyrie_B">
 	<xacro:property name="instance" value="valkyrie_B" />
-	<xacro:include filename="$(find val_description)/common/xacro/serial_numbers/valkyrie_B_serials.xacro" />
-    <xacro:include filename="$(find val_description)/instance/instances/robots/xacro/common/valkyrie_full_template.xacro"/>
+	<xacro:include filename="../../../common/xacro/serial_numbers/valkyrie_B_serials.xacro" />
+    <xacro:include filename="../../../instance/instances/robots/xacro/common/valkyrie_full_template.xacro"/>
 </robot>

File: instance/instances/robots/valkyrie_C.xacro (robot description, xacro)
@@ -1,5 +1,5 @@
 <robot xmlns:xacro="http://www.ros.org/wiki/xacro" name="valkyrie_C">
 	<xacro:property name="instance" value="valkyrie_C" />
-	<xacro:include filename="$(find val_description)/common/xacro/serial_numbers/valkyrie_C_serials.xacro" />
-    <xacro:include filename="$(find val_description)/instance/instances/robots/xacro/common/valkyrie_full_template.xacro"/>
+	<xacro:include filename="../../../common/xacro/serial_numbers/valkyrie_C_serials.xacro" />
+    <xacro:include filename="../../../instance/instances/robots/xacro/common/valkyrie_full_template.xacro"/>
 </robot>

File: instance/instances/robots/valkyrie_D.xacro (robot description, xacro)
@@ -1,5 +1,5 @@
 <robot xmlns:xacro="http://www.ros.org/wiki/xacro" name="valkyrie_D">
     <xacro:property name="instance" value="valkyrie_D" />
-    <xacro:include filename="$(find val_description)/common/xacro/serial_numbers/valkyrie_D_serials.xacro" />
-    <xacro:include filename="$(find val_description)/instance/instances/robots/xacro/common/valkyrie_full_template.xacro"/>
+    <xacro:include filename="../../../common/xacro/serial_numbers/valkyrie_D_serials.xacro" />
+    <xacro:include filename="../../../instance/instances/robots/xacro/common/valkyrie_full_template.xacro"/>
 </robot>

File: instance/instances/robots/valkyrie_E.xacro (robot description, xacro)
@@ -1,5 +1,5 @@
 <robot xmlns:xacro="http://www.ros.org/wiki/xacro" name="valkyrie_E">
 	<xacro:property name="instance" value="valkyrie_E" />
-	<xacro:include filename="$(find val_description)/common/xacro/serial_numbers/valkyrie_E_serials.xacro" />
-    <xacro:include filename="$(find val_description)/instance/instances/robots/xacro/common/valkyrie_full_template.xacro"/>
+	<xacro:include filename="../../../common/xacro/serial_numbers/valkyrie_E_serials.xacro" />
+    <xacro:include filename="../../../instance/instances/robots/xacro/common/valkyrie_full_template.xacro"/>
 </robot>

File: instance/instances/robots/xacro/common/test_bench_template.xacro (robot description, xacro)
@@ -1,7 +1,7 @@
 <robot xmlns:xacro="http://www.ros.org/wiki/xacro" name="test_bench_template">
-	<xacro:include filename="$(find val_description)/common/xacro/serial_numbers/test_bench_serials.xacro" />
-	<xacro:include filename="$(find val_description)/common/xacro/nodes/actuator_testbench_nodes.xacro" />
-	<xacro:include filename="$(find val_description)/instance/instances/robots/xacro/mechanisms/mechanisms.xacro"/>
-	<xacro:include filename="$(find val_description)/common/xacro/firmware/valkyrie_firmware.xacro"/>
+	<xacro:include filename="../../../../../common/xacro/serial_numbers/test_bench_serials.xacro" />
+	<xacro:include filename="../../../../../common/xacro/nodes/actuator_testbench_nodes.xacro" />
+	<xacro:include filename="../../../../../instance/instances/robots/xacro/mechanisms/mechanisms.xacro"/>
+	<xacro:include filename="../../../../../common/xacro/firmware/valkyrie_firmware.xacro"/>
 	<RobotInstance id="testbench" />
 	<Channels>

File: instance/instances/robots/xacro/common/valkyrie_full_template.xacro (robot description, xacro)
@@ -1,12 +1,12 @@
 <robot xmlns:xacro="http://www.ros.org/wiki/xacro" name="valkyrie_template">
-	<xacro:include filename="$(find val_description)/common/xacro/nodes/valkyrie_nodes.xacro" />
-	<xacro:include filename="$(find val_description)/instance/instances/robots/xacro/limbs/leg/leg.xacro" />
-	<xacro:include filename="$(find val_description)/instance/instances/robots/xacro/limbs/arm/arm.xacro" />
-	<xacro:include filename="$(find val_description)/instance/instances/robots/xacro/limbs/neck/neck.xacro" />
-	<xacro:include filename="$(find val_description)/instance/instances/robots/xacro/limbs/waist/waist.xacro" />
-	<xacro:include filename="$(find val_description)/instance/instances/robots/xacro/sensors/imu.xacro" />
-	<xacro:include filename="$(find val_description)/instance/instances/robots/xacro/sensors/ati_force_torque.xacro" />
-	<xacro:include filename="$(find val_description)/instance/instances/robots/xacro/firmware/firmware.xacro" />
-	<xacro:include filename="$(find val_description)/instance/instances/robots/xacro/common/joint_calibration_angles.xacro" />
+	<xacro:include filename="../../../../../common/xacro/nodes/valkyrie_nodes.xacro" />
+	<xacro:include filename="../../../../../instance/instances/robots/xacro/limbs/leg/leg.xacro" />
+	<xacro:include filename="../../../../../instance/instances/robots/xacro/limbs/arm/arm.xacro" />
+	<xacro:include filename="../../../../../instance/instances/robots/xacro/limbs/neck/neck.xacro" />
+	<xacro:include filename="../../../../../instance/instances/robots/xacro/limbs/waist/waist.xacro" />
+	<xacro:include filename="../../../../../instance/instances/robots/xacro/sensors/imu.xacro" />
+	<xacro:include filename="../../../../../instance/instances/robots/xacro/sensors/ati_force_torque.xacro" />
+	<xacro:include filename="../../../../../instance/instances/robots/xacro/firmware/firmware.xacro" />
+	<xacro:include filename="../../../../../instance/instances/robots/xacro/common/joint_calibration_angles.xacro" />
 	<RobotInstance id="${instance}" />
 	<xacro:all_channels/>

File: instance/instances/robots/xacro/firmware/arm_firmware.xacro (robot description, xacro)
@@ -1,4 +1,4 @@
 <robot xmlns:xacro="http://www.ros.org/wiki/xacro" name="arm_firmware">
-    <xacro:include filename="$(find val_description)/common/xacro/firmware/valkyrie_firmware.xacro"/>
+    <xacro:include filename="../../../../../common/xacro/firmware/valkyrie_firmware.xacro"/>
     <xacro:macro name="arm_firmware"  >
             <fw id="rightArmJ1">

File: instance/instances/robots/xacro/firmware/firmware.xacro (robot description, xacro)
@@ -1,9 +1,13 @@
-<firmware xmlns:xacro="http://www.ros.org/wiki/xacro" name="firmware">
-    <xacro:include filename="$(find val_description)/instance/instances/robots/xacro/firmware/arm_firmware.xacro" />
-    <xacro:include filename="$(find val_description)/instance/instances/robots/xacro/firmware/forearm_firmware.xacro" />
-    <xacro:include filename="$(find val_description)/instance/instances/robots/xacro/firmware/leg_firmware.xacro" />
-    <xacro:include filename="$(find val_description)/instance/instances/robots/xacro/firmware/trunk_firmware.xacro" />
-    <xacro:include filename="$(find val_description)/common/xacro/firmware/valkyrie_firmware.xacro"/>
+<robot xmlns:xacro="http://www.ros.org/wiki/xacro" name="firmware">
+    <xacro:include filename="../../../../../instance/instances/robots/xacro/firmware/arm_firmware.xacro" />
+    <xacro:include filename="../../../../../instance/instances/robots/xacro/firmware/forearm_firmware.xacro" />
+    <xacro:include filename="../../../../../instance/instances/robots/xacro/firmware/leg_firmware.xacro" />
+    <xacro:include filename="../../../../../instance/instances/robots/xacro/firmware/trunk_firmware.xacro" />
     <xacro:macro name="firmware" params="">
+<!--
+    There is a bug in xacro that is causing it not to resolve global-scope properties unless I add a
+    local property here. The name of the property apparently doesn't matter.
+-->
+        <xacro:property name="foo" value="bar" />
         <Firmware type="firmware">
             <xacro:arm_firmware />
@@ -13,3 +17,3 @@
         </Firmware>
     </xacro:macro>
-</firmware>
+</robot>

File: instance/instances/robots/xacro/firmware/forearm_firmware.xacro (robot description, xacro)
@@ -1,4 +1,4 @@
 <robot xmlns:xacro="http://www.ros.org/wiki/xacro" name="forearm_firmware">
-    <xacro:include filename="$(find val_description)/common/xacro/firmware/valkyrie_firmware.xacro"/>
+    <xacro:include filename="../../../../../common/xacro/firmware/valkyrie_firmware.xacro"/>
     <xacro:macro name="forearm_firmware"  >
             <fw id="leftArmJ5">

File: instance/instances/robots/xacro/limbs/arm/arm.xacro (robot description, xacro)
@@ -1,5 +1,5 @@
 <robot xmlns:xacro="http://www.ros.org/wiki/xacro" name="arm">
-    <xacro:include filename="$(find val_description)/instance/instances/robots/xacro/mechanisms/mechanisms.xacro"/>
-    <xacro:include filename="$(find val_description)/common/xacro/joint_names/valkyrie_joint_names.xacro"/>
+    <xacro:include filename="../../../../../../instance/instances/robots/xacro/mechanisms/mechanisms.xacro"/>
+    <xacro:include filename="../../../../../../common/xacro/joint_names/valkyrie_joint_names.xacro"/>
     <xacro:macro name="arm" params="prefix reflect j1_serial_number j2_serial_number j3_serial_number j4_serial_number j5_serial_number forearm_serial_number" >
     	<xacro:simple_mechanism name="${ShoulderPitchJointName}" serial_number="${j1_serial_number}" node="/trunk/${prefix}_arm_j1" calibration_angle="${ShoulderPitchCalibrationAngle}"/>

File: instance/instances/robots/xacro/limbs/leg/leg.xacro (robot description, xacro)
@@ -1,5 +1,5 @@
 <robot xmlns:xacro="http://www.ros.org/wiki/xacro" name="leg">
-    <xacro:include filename="$(find val_description)/instance/instances/robots/xacro/mechanisms/mechanisms.xacro"/>
-    <xacro:include filename="$(find val_description)/common/xacro/joint_names/valkyrie_joint_names.xacro"/>
+    <xacro:include filename="../../../../../../instance/instances/robots/xacro/mechanisms/mechanisms.xacro"/>
+    <xacro:include filename="../../../../../../common/xacro/joint_names/valkyrie_joint_names.xacro"/>
     <xacro:macro name="leg" params="prefix reflect j1_serial_number j2_serial_number j3_serial_number j4_serial_number ankle_left_actuator_serial ankle_right_actuator_serial" >
     	<xacro:simple_mechanism name="${HipYawJointName}" serial_number="${j1_serial_number}" node="/pelvis/${prefix}_leg_j1" calibration_angle="${HipYawCalibrationAngle}"/>

File: instance/instances/robots/xacro/limbs/neck/neck.xacro (robot description, xacro)
@@ -1,5 +1,5 @@
 <robot xmlns:xacro="http://www.ros.org/wiki/xacro" name="neck">
-    <xacro:include filename="$(find val_description)/instance/instances/robots/xacro/mechanisms/mechanisms.xacro"/>
-    <xacro:include filename="$(find val_description)/common/xacro/joint_names/valkyrie_joint_names.xacro"/>
+    <xacro:include filename="../../../../../../instance/instances/robots/xacro/mechanisms/mechanisms.xacro"/>
+    <xacro:include filename="../../../../../../common/xacro/joint_names/valkyrie_joint_names.xacro"/>
     <xacro:macro name="neck" params="j1_serial_number j2_serial_number j3_serial_number" >
     	<xacro:simple_mechanism name="${LowerNeckPitchJointName}" serial_number="${j1_serial_number}" node="${LowerNeckPitchNode}" calibration_angle="${LowerNeckPitchCalibrationAngle}"/>

File: instance/instances/robots/xacro/limbs/waist/waist.xacro (robot description, xacro)
@@ -1,6 +1,6 @@
 <robot xmlns:xacro="http://www.ros.org/wiki/xacro" name="waist">
-    <xacro:include filename="$(find val_description)/instance/instances/robots/xacro/mechanisms/mechanisms.xacro"/>
-    <xacro:include filename="$(find val_description)/common/xacro/joint_names/valkyrie_joint_names.xacro"/>
-    <xacro:include filename="$(find val_description)/common/xacro/actuator_names/valkyrie_actuator_names.xacro"/>
+    <xacro:include filename="../../../../../../instance/instances/robots/xacro/mechanisms/mechanisms.xacro"/>
+    <xacro:include filename="../../../../../../common/xacro/joint_names/valkyrie_joint_names.xacro"/>
+    <xacro:include filename="../../../../../../common/xacro/actuator_names/valkyrie_actuator_names.xacro"/>
     <xacro:macro name="waist" params="j1_serial_number waist_left_actuator_serial waist_right_actuator_serial" >
     	<xacro:simple_mechanism name="${TorsoYawJointName}" serial_number="${j1_serial_number}" node="${TrunkYawNode}" calibration_angle="${TorsoYawCalibrationAngle}"/>

File: model/robots/common/xacro/arm/arm_includes.xacro (robot description, xacro)
@@ -1,11 +1,11 @@
 <robot xmlns:xacro="http://www.ros.org/wiki/xacro" name="arm_includes">
-	<xacro:include filename="$(find val_description)/model/robots/common/xacro/arm/joint_axes.xacro"/>
-	<xacro:include filename="$(find val_description)/model/robots/common/xacro/arm/joint_limits.xacro"/>
-	<xacro:include filename="$(find val_description)/model/robots/common/xacro/arm/frame_parameters.xacro"/>
-	<xacro:include filename="$(find val_description)/model/robots/common/xacro/arm/mass_parameters.xacro"/>
-	<xacro:include filename="$(find val_description)/common/xacro/joint_names/valkyrie_joint_names.xacro"/>
-	<xacro:include filename="$(find val_description)/common/xacro/actuator_names/valkyrie_actuator_names.xacro"/>
-	<xacro:include filename="$(find val_description)/model/robots/common/xacro/gains${robot_type_suffix}.xacro"/>
-	<xacro:include filename="$(find val_description)/model/robots/common/xacro/gazebo_hand_contact.xacro"/>
-	<xacro:include filename="$(find val_description)/model/robots/common/xacro/arm/arm.xacro"/>
+	<xacro:include filename="joint_axes.xacro"/>
+	<xacro:include filename="joint_limits.xacro"/>
+	<xacro:include filename="frame_parameters.xacro"/>
+	<xacro:include filename="mass_parameters.xacro"/>
+	<xacro:include filename="../../../../../common/xacro/joint_names/valkyrie_joint_names.xacro"/>
+	<xacro:include filename="../../../../../common/xacro/actuator_names/valkyrie_actuator_names.xacro"/>
+	<xacro:include filename="../../../../../model/robots/common/xacro/gains${robot_type_suffix}.xacro"/>
+	<xacro:include filename="../../../../../model/robots/common/xacro/gazebo_hand_contact.xacro"/>
+	<xacro:include filename="arm.xacro"/>
 </robot>

File: model/robots/common/xacro/common_bodies.xacro (robot description, xacro)
@@ -1,6 +1,6 @@
 <robot xmlns:xacro="http://www.ros.org/wiki/xacro" name="common_bodies">
-    <xacro:include filename="$(find val_description)/model/robots/common/xacro/index_finger/index_finger.xacro" />
-    <xacro:include filename="$(find val_description)/model/robots/common/xacro/middle_finger/middle_finger.xacro" />
-    <xacro:include filename="$(find val_description)/model/robots/common/xacro/pinky_finger/pinky_finger.xacro" />
-    <xacro:include filename="$(find val_description)/model/robots/common/xacro/thumb/thumb.xacro" />
+    <xacro:include filename="index_finger/index_finger.xacro" />
+    <xacro:include filename="middle_finger/middle_finger.xacro" />
+    <xacro:include filename="pinky_finger/pinky_finger.xacro" />
+    <xacro:include filename="thumb/thumb.xacro" />
 </robot>

File: model/robots/common/xacro/gains_sim.xacro (robot description, xacro)
@@ -1,5 +1,5 @@
 <robot xmlns:xacro="http://www.ros.org/wiki/xacro" name="valkyrie_nodes">
     <!-- Get the hardware gains -->
-    <xacro:include filename="$(find val_description)/model/robots/common/xacro/gains.xacro"/>
+    <xacro:include filename="gains.xacro"/>
     <!-- Override only those properties that need to be different for sim -->
     <xacro:property name="LowerNeckPitchKp" value="150" />
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