Commit message: add Zedm model to the valkyrie URDFs. sim and visual urdfs have the complete model. the hw urdfs only have the zedm_mount transform.

File: model/robots/common/xacro/head/head.xacro (robot description, xacro)
@@ -62,4 +62,16 @@
       <xacro:fixed_joint jointName="multisense_head_root_joint" parent="upperNeckPitchLink" child="multisense/head" origin_xyz="0.183585961 0.0 0.075353826" origin_rpy="-3.14159 0.130899694 0.0" />
     </xacro:macro>
+    <xacro:macro name="include_zedm_sim">
+      <xacro:massless_virtual_link name="zedm_mount" origin_xyz="0 0 0" origin_rpy="0 0 0"/>
+      <xacro:fixed_joint jointName="zedm_head_root_joint" parent="upperNeckPitchLink" child="zedm_mount" origin_xyz="0.192184 0.0 -0.096498" origin_rpy="0.0 0.1309 0.0" />
+      <xacro:include filename="$(find val_description)/model/urdf/zed/zed_macro.urdf.xacro" />
+      <xacro:zed_camera name="zedm" model="zedm" parent="zedm_mount">
+        <origin xyz="0.0 0.0 0.0" rpy="0.0 0.0 0.0" />
+      </xacro:zed_camera>
+    </xacro:macro>
+    <xacro:macro name="include_zedm_hw">
+      <xacro:massless_virtual_link name="zedm_mount" origin_xyz="0 0 0" origin_rpy="0 0 0"/>
+      <xacro:fixed_joint jointName="zedm_head_root_joint" parent="upperNeckPitchLink" child="zedm_mount" origin_xyz="0.192184 0.0 -0.096498" origin_rpy="0.0 0.1309 0.0" />
+    </xacro:macro>
     <xacro:macro name="neck_transmissions_hw">
       <xacro:simple_position_transmission jointName="${LowerNeckPitchJointName}" actuatorName="${LowerNeckPitchActuatorName}" nodeName="${LowerNeckPitchNode}" actuatorApi="${LowerNeckPitchApi}"/>

File: model/robots/common/xacro/valkyrie_arm_mass_sims_base_hw.xacro (robot description, xacro)
@@ -11,4 +11,5 @@
     <xacro:v1_leg_sensors prefix="right" reflect="-1" ATI_serial_number="${right_foot_ATI_serial}" ATI_node="${right_foot_ATI_node}"/>
     <xacro:include_multisense_hw />
+    <xacro:include_zedm_hw />
     <xacro:v1_pelvis_rear_sensors_usb sensor_node_tag="${pelvis_rear_imu_node}" sensor_api_tag="${ImuMicrostrainHardwareApi}"  sensor_port_tag="${pelvis_rear_imu_port}"/>
     <xacro:waist_transmissions_hw />

File: model/robots/common/xacro/valkyrie_arm_mass_sims_base_sim.xacro (robot description, xacro)
@@ -11,4 +11,5 @@
     <xacro:v1_leg_sensors prefix="right" reflect="-1" ATI_serial_number="${sim_ATI_serial}" ATI_node="${right_foot_ATI_node}"/>
     <xacro:include_multisense_sim />
+    <xacro:include_zedm_sim />
     <xacro:v1_trunk_sensors_usb sensor_node_tag="${torso_left_imu_node}" sensor_api_tag="${ImuSensorSimApi}" sensor_port_tag="${torso_left_imu_port}"/>
     <xacro:waist_transmissions_sim />

File: model/robots/common/xacro/valkyrie_base_hw.xacro (robot description, xacro)
@@ -19,4 +19,5 @@
     <xacro:v1_leg_sensors prefix="right" reflect="-1" ATI_serial_number="${right_foot_ATI_serial}" ATI_node="${right_foot_ATI_node}"/>
     <xacro:include_multisense_hw />
+    <xacro:include_zedm_hw />
     <xacro:v1_pelvis_rear_sensors_usb sensor_node_tag="${pelvis_rear_imu_node}" sensor_api_tag="${ImuMicrostrainHardwareApi}"  sensor_port_tag="${pelvis_rear_imu_port}"/>
     <xacro:waist_transmissions_hw />

File: model/robots/common/xacro/valkyrie_base_sim.xacro (robot description, xacro)
@@ -19,4 +19,5 @@
     <xacro:v1_leg_sensors prefix="right" reflect="-1" ATI_serial_number="${sim_ATI_serial}" ATI_node="${right_foot_ATI_node}"/>
     <xacro:include_multisense_sim />
+    <xacro:include_zedm_sim />
     <xacro:v1_trunk_sensors_usb sensor_node_tag="${torso_left_imu_node}" sensor_api_tag="${ImuSensorSimApi}" sensor_port_tag="${torso_left_imu_port}"/>
     <xacro:waist_transmissions_sim />

File: model/robots/common/xacro/valkyrie_imu_base.xacro (robot description, xacro)
@@ -3,4 +3,5 @@
     <xacro:make_pelvis />
     <xacro:include_multisense_hw />
+    <xacro:include_zedm_hw />
     <xacro:v1_pelvis_middle_sensors_usb sensor_node_tag="${pelvis_middle_imu_node}" sensor_api_tag="${KVHHardwareApi}"  sensor_port_tag="${pelvis_middle_imu_port}"/>
 </robot>

File: model/robots/common/xacro/valkyrie_simple_base.xacro (robot description, xacro)
@@ -19,4 +19,5 @@
     <xacro:v1_leg_sensors prefix="right" reflect="-1" ATI_serial_number="${sim_ATI_serial}" ATI_node="${right_foot_ATI_node}"/>
     <xacro:include_multisense_sim />
+    <xacro:include_zedm_sim />
     <xacro:v1_trunk_sensors_usb sensor_node_tag="${torso_left_imu_node}" sensor_api_tag="${ImuSensorSimApi}" sensor_port_tag="${torso_left_imu_port}"/>
 </robot>

Commit message: modify multisense_sl.urdf to change the joint name. also, include missing multisense tf frames.

File: model/robots/common/xacro/head/head.xacro (robot description, xacro)
@@ -57,6 +57,5 @@
     <xacro:macro name="include_multisense_sim">
       <xacro:fixed_joint jointName="multisense_head_root_joint" parent="upperNeckPitchLink" child="multisense/head" origin_xyz="0.183585961 0.0 0.075353826" origin_rpy="-3.14159 0.130899694 0.0" />
-      <xacro:include filename="$(find val_description)/model/urdf/multisense_sl/multisenseSL.urdf.xacro" />
-      <xacro:multisenseSL name="multisense" />
+      <xacro:include filename="$(find val_description)/model/urdf/multisense_sl.urdf" />
     </xacro:macro>
     <xacro:macro name="include_multisense_hw">

File: model/urdf/multisense_sl.urdf (robot description, URDF)
Before this commit: robot multisense_sl, 11 links, 10 joints
Links:
- added link multisense/accel
- added link multisense/gyro
- added link multisense/mag
Joints:
- removed joint hokuyo_joint
- added joint multisense/accel_joint: type fixed, parent multisense/head, child multisense/accel, origin xyz=-.0475 .0302 -.00275 rpy=0 1.5707 0
- added joint multisense/gyro_joint: type fixed, parent multisense/head, child multisense/gyro, origin xyz=-.0476 .0388 -.00075 rpy=1.5707 3.14159 1.5707 
- added joint multisense/mag_joint: type fixed, parent multisense/head, child multisense/mag, origin xyz=-.0475 .0302 -.00275 rpy=0 1.5707 0
- added joint multisense/motor_joint: type continuous, parent multisense/head, child multisense/hokuyo_link, origin xyz=-0.0446 0 0.0880 rpy=0 0 0, axis 1 0 0
