Commit message: Convert A to using PCI-based IMUs

File: common/xacro/dev_ports/valkyrie_A_ports.xacro (robot description, xacro)
@@ -1,5 +1,5 @@
 <robot xmlns:xacro="http://www.ros.org/wiki/xacro" name="valkyrie_A_ports">
 	<xacro:property name="pelvis_middle_imu_port" value="/dev/ttyACM0" />
-	<xacro:property name="pelvis_rear_imu_port" value="/dev/serial/by-id/usb-Lord_Microstrain_Lord_Inertial_Sensor_0000__6233.47095-if00" />
-	<xacro:property name="torso_left_imu_port" value="/dev/serial/by-id/usb-Lord_Microstrain_Lord_Inertial_Sensor_0000__6233.47090-if00" />
+	<xacro:property name="pelvis_rear_imu_port" value="/dev/ttyF3" />
+	<xacro:property name="torso_left_imu_port" value="/dev/ttyF0" />
 </robot>

Commit message: IMU serial ports for Val A

File: common/xacro/dev_ports/valkyrie_A_ports.xacro (robot description, xacro)
@@ -1,5 +1,5 @@
 <robot xmlns:xacro="http://www.ros.org/wiki/xacro" name="valkyrie_A_ports">
 	<xacro:property name="pelvis_middle_imu_port" value="/dev/ttyACM0" />
-	<xacro:property name="pelvis_rear_imu_port" value="/dev/ttyF3" />
-	<xacro:property name="torso_left_imu_port" value="/dev/ttyF0" />
+	<xacro:property name="pelvis_rear_imu_port" value="/dev/ttyS4" />
+	<xacro:property name="torso_left_imu_port" value="/dev/ttyS5" />
 </robot>
