Commit message: Swap in Val-C IMU #47250 to Val-B

File: common/xacro/dev_ports/valkyrie_B_ports.xacro (robot description, xacro)
@@ -4,4 +4,7 @@
   <!-- <xacro:property name="pelvis_rear_imu_port" value="/dev/serial/by-id/usb-Lord_Microstrain_Lord_Inertial_Sensor_0000__6233.47099-if00" /> -->
   <xacro:property name="pelvis_rear_imu_port" value="/dev/serial/by-id/usb-Lord_Microstrain_Lord_Inertial_Sensor_0000__6233.47092-if00" />
-	<xacro:property name="torso_left_imu_port" value="/dev/serial/by-id/usb-Lord_Microstrain_Lord_Inertial_Sensor_0000__6233.47097-if00" />
+        <!-- Original chest IMU on B -->
+	<!--xacro:property name="torso_left_imu_port" value="/dev/serial/by-id/usb-Lord_Microstrain_Lord_Inertial_Sensor_0000__6233.47097-if00" /-->
+        <!-- Chest IMU swapped in from C -->
+	<xacro:property name="torso_left_imu_port" value="/dev/serial/by-id/usb-Lord_Microstrain_Lord_Inertial_Sensor_0000__6233.47250-if00" />
 </robot>

Commit message: Change USB IMU ports to serial

File: common/xacro/dev_ports/valkyrie_B_ports.xacro (robot description, xacro)
@@ -1,10 +1,5 @@
 <robot xmlns:xacro="http://www.ros.org/wiki/xacro" name="valkyrie_B_ports">
-	<xacro:property name="pelvis_middle_imu_port" value="/dev/serial/by-id/usb-Lord_Microstrain_Lord_Inertial_Sensor_0000__6233.47094-if00" />
-	<!-- <xacro:property name="pelvis_rear_imu_port" value="/dev/serial/by-id/usb-FTDI_USB-RS232_Cable_FTY5H9NH-if00-port0" /> -->
-  <!-- <xacro:property name="pelvis_rear_imu_port" value="/dev/serial/by-id/usb-Lord_Microstrain_Lord_Inertial_Sensor_0000__6233.47099-if00" /> -->
-  <xacro:property name="pelvis_rear_imu_port" value="/dev/serial/by-id/usb-Lord_Microstrain_Lord_Inertial_Sensor_0000__6233.47092-if00" />
-        <!-- Original chest IMU on B -->
-	<!--xacro:property name="torso_left_imu_port" value="/dev/serial/by-id/usb-Lord_Microstrain_Lord_Inertial_Sensor_0000__6233.47097-if00" /-->
-        <!-- Chest IMU swapped in from C -->
-	<xacro:property name="torso_left_imu_port" value="/dev/serial/by-id/usb-Lord_Microstrain_Lord_Inertial_Sensor_0000__6233.47250-if00" />
+	<xacro:property name="pelvis_middle_imu_port" value="/dev/ttyACM0" />
+	<xacro:property name="pelvis_rear_imu_port" value="/dev/ttyF3" />
+	<xacro:property name="torso_left_imu_port" value="/dev/ttyF0" />
 </robot>

Commit message: Switch B to new serial card config

File: common/xacro/dev_ports/valkyrie_B_ports.xacro (robot description, xacro)
@@ -1,5 +1,5 @@
 <robot xmlns:xacro="http://www.ros.org/wiki/xacro" name="valkyrie_B_ports">
 	<xacro:property name="pelvis_middle_imu_port" value="/dev/ttyACM0" />
-	<xacro:property name="pelvis_rear_imu_port" value="/dev/ttyF3" />
-	<xacro:property name="torso_left_imu_port" value="/dev/ttyF0" />
+	<xacro:property name="pelvis_rear_imu_port" value="/dev/ttyS4" />
+	<xacro:property name="torso_left_imu_port" value="/dev/ttyS5" />
 </robot>
