Commit message: Updates to valkyrie_nodes.xacro

File: common/xacro/nodes/forearm_testbench_nodes.xacro (robot description, xacro)
@@ -2,11 +2,11 @@
 	<xacro:property name="HandSensorNode" value="_arm/forearm_sensors"/>
     <xacro:property name="testbench_node" value="/right_arm/j5" />
-    <xacro:property name="IndexNode" value="_arm/hand/index" />
-    <xacro:property name="MiddleNode" value="_arm/hand/middle" />
-    <xacro:property name="PinkyNode" value="_arm/hand/pinky" />
-    <xacro:property name="ThumbProxNode" value="_arm/hand/thumb_proximal" />
-    <xacro:property name="ThumbDistNode" value="_arm/hand/thumb_distal" />
+    <xacro:property name="IndexFingerNode" value="_arm/hand/index" />
+    <xacro:property name="MiddleFingerNode" value="_arm/hand/middle" />
+    <xacro:property name="PinkyFingerNode" value="_arm/hand/pinky" />
+    <xacro:property name="ThumbProximalNode" value="_arm/hand/thumb_proximal" />
+    <xacro:property name="ThumbDistalNode" value="_arm/hand/thumb_distal" />
     <xacro:property name="ThumbRollNode" value="_arm/hand/thumb_roll" />
-    <xacro:property name="WristLeftNode" value="_arm/wrist/left_actuator" />
-    <xacro:property name="WristRightNode" value="_arm/wrist/right_actuator" />
+    <xacro:property name="WristLeftActuatorNode" value="_arm/wrist/left_actuator" />
+    <xacro:property name="WristRightActuatorNode" value="_arm/wrist/right_actuator" />
 </robot>

File: common/xacro/nodes/valkyrie_nodes.xacro (robot description, xacro)
@@ -1,4 +1,4 @@
 <robot xmlns:xacro="http://www.ros.org/wiki/xacro" name="valkyrie_nodes">
-	<!--<xacro:property name="HipYawNode" value="/pelvis/${prefix}_leg_j1" /> -->
+	<xacro:property name="HipYawNode" value="_leg_j1" />
 	<xacro:property name="HipRollNode" value="_leg/j2" />
 	<xacro:property name="HipPitchNode" value="_leg/j3" />
@@ -6,20 +6,11 @@
 	<xacro:property name="AnkleLeftActuatorNode" value="_leg/ankle/left_actuator" />
 	<xacro:property name="AnkleRightActuatorNode" value="_leg/ankle/right_actuator" />
-	<xacro:property name="ShoulderPitchNode" value="/trunk/${prefix}_arm_j1" />
+	<xacro:property name="ShoulderPitchNode" value="_arm_j1" />
 	<xacro:property name="ShoulderRollNode" value="_arm/j2" />
 	<xacro:property name="ShoulderYawNode" value="_arm/j3" />
 	<xacro:property name="ElbowPitchNode" value="_arm/j4" />
 	<xacro:property name="ForearmYawNode" value="_arm/j5" />
-	<xacro:property name="WristTopActuatorNode" value="_arm/wrist/top_actautor" />
-	<xacro:property name="WristBottomActuatorNode" value="_arm/wrist/bottom_actuator" />
 	<xacro:property name="WristLeftActuatorNode" value="_arm/wrist/left_actuator" />
 	<xacro:property name="WristRightActuatorNode" value="_arm/wrist/right_actuator" />
-    	<xacro:property name="IndexNode" value="_arm/hand/index" />
-    	<xacro:property name="MiddleNode" value="_arm/hand/middle" />
-    	<xacro:property name="PinkyNode" value="_arm/hand/pinky" />
-    	<xacro:property name="ThumbProxNode" value="_arm/hand/thumb_proximal" />
-    	<xacro:property name="ThumbDistNode" value="_arm/hand/thumb_distal" />
-    	<xacro:property name="WristLeftNode" value="_arm/wrist/left_actuator" />
-    	<xacro:property name="WristRightNode" value="_arm/wrist/right_actuator" />
 	<xacro:property name="LowerNeckPitchNode" value="/neck/j1" />
 	<xacro:property name="NeckYawNode" value="/neck/j2" />
@@ -28,6 +19,4 @@
 	<xacro:property name="WaistLeftActuatorNode" value="/trunk/left_actuator" /> <!--pitch-->
 	<xacro:property name="WaistRightActuatorNode" value="/trunk/right_actuator" /> <!--roll-->
-	<xacro:property name="Athena1Node" value="/${prefix}_arm/athena1"/>
-	<xacro:property name="Athena2Node" value="/${prefix}_arm/athena2"/>
 	<xacro:property name="pelvis_middle_imu_node" value="/sensors/middlePelvisIMU" />
 	<xacro:property name="pelvis_rear_imu_node" value="/sensors/rearPelvisIMU" />
@@ -55,15 +44,60 @@
 	<xacro:property name="ThumbPitch2Node" value="_arm/forearm_sensors/thumb"/>
 	<xacro:property name="ThumbPitch3Node" value="_arm/forearm_sensors/thumb"/>
-	<xacro:macro name="all_channels" >
-		<Channels>
-			<Channel id="/right_arm" address="1" />
-			<Channel id="/left_arm" address="5" />
-			<Channel id="/right_leg" address="4" />
-			<Channel id="/left_leg" address="6" />
-			<Channel id="/neck" address="0" />
-			<Channel id="/trunk" address="7" />
-			<Channel id="/power" address="2" />
-			<Channel id="/pelvis" address="3" />
-		</Channels>
+    <xacro:macro name="robonet_arm_channel_nodes">
+        <Node id="forearm_sensors" address="1"/>
+        <Node id="j2" address="2"/>
+        <Node id="j3" address="3"/>
+        <Node id="j4" address="4"/>
+        <Node id="j5" address="5"/>
+        <Node id="hand/index" address="6"/>
+        <Node id="hand/pinky" address="7"/>
+        <Node id="hand/thumb_distal" address="8"/>
+        <Node id="hand/middle" address="9"/>
+        <Node id="hand/thumb_roll" address="10"/>
+        <Node id="wrist/left_actuator" address="11"/>
+        <Node id="hand/thumb_proximal" address="12"/>
+        <Node id="wrist/right_actuator" address="13"/>
+    </xacro:macro>
+    <xacro:macro name="robonet_leg_channel_nodes">
+        <Node id="j2" address="2"/>
+        <Node id="j3" address="3"/>
+        <Node id="j4" address="4"/>
+        <Node id="ankle/right_actuator" address="5"/>
+        <Node id="ankle/left_actuator" address="6"/>
+    </xacro:macro>
+	<xacro:macro name="robonet_config" >
+		<RobonetConfig>
+			<Channel id="/right_arm" address="1">
+                <xacro:robonet_arm_channel_nodes/>
+            </Channel>
+			<Channel id="/left_arm" address="5">
+                <xacro:robonet_arm_channel_nodes/>
+            </Channel>
+			<Channel id="/right_leg" address="4">
+                <xacro:robonet_leg_channel_nodes/>
+            </Channel>
+			<Channel id="/left_leg" address="6">
+                <xacro:robonet_leg_channel_nodes/>
+            </Channel>
+			<Channel id="/neck" address="0">
+                <Node id="j1" address="1"/>
+                <Node id="j2" address="2"/>
+                <Node id="j3" address="3"/>
+            </Channel>
+			<Channel id="/trunk" address="7">
+                <Node id="left_arm_j1" address="1"/>
+                <Node id="left_actuator" address="2"/>
+                <Node id="right_actuator" address="3"/>
+                <Node id="right_arm_j1" address="4"/>
+            </Channel>
+			<Channel id="/power" address="2">
+                <Node id="pdbmti" address="1"/>
+            </Channel>
+			<Channel id="/pelvis" address="3">
+                <Node id="waist" address="1"/>
+                <Node id="left_leg_j1" address="3"/>
+                <Node id="right_leg_j1" address="5"/>
+            </Channel>
+		</RobonetConfig>
 	</xacro:macro>
 </robot>

File: common/xacro/nodes/valkyrie_sim_nodes.xacro (robot description, xacro)
@@ -45,5 +45,5 @@
 	<xacro:property name="PinkyPitch2Node" value="_hand/pinky_pitch_2"/>
 	<xacro:property name="PinkyPitch3Node" value="_hand/pinky_pitch_3"/>
-	<xacro:macro name="all_channels" >
+	<xacro:macro name="robonet_config" >
 		<Channels>
 			<Channel id="/right_arm" />

File: instance/instances/robots/forearm_testbench_left.xacro (robot description, xacro)
@@ -3,5 +3,5 @@
 	<xacro:property name="prefix" value="left" />
     <xacro:include filename="../../../common/xacro/firmware/valkyrie_firmware.xacro"/>
-	<xacro:include filename="../../../common/xacro/nodes/forearm_testbench_nodes_left.xacro" />
+	<xacro:include filename="../../../common/xacro/nodes/forearm_testbench_nodes.xacro" />
 	<xacro:include filename="../../../common/xacro/serial_numbers/forearm_testbench_serials.xacro" />
     <xacro:include filename="../../../instance/instances/robots/xacro/mechanisms/mechanisms.xacro"/>

File: instance/instances/robots/forearm_testbench_right.xacro (robot description, xacro)
@@ -13,5 +13,5 @@
     <Mechanisms>
     <xacro:simple_mechanism name="testbench_actuator" serial_number="${forearm_yaw_serial_number}" node="${testbench_node}" />
-    <xacro:hand_mechanism mechanism_name="${prefix}Hand" serial_number="${hand_serial_number}" index_node="/${prefix}${IndexNode}" middle_node="/${prefix}${MiddleNode}" pinky_node="/${prefix}${PinkyNode}" thumb_prox_node="/${prefix}${ThumbProxNode}" thumb_dist_node="/${prefix}${ThumbDistNode}" thumb_roll_node="/${prefix}${ThumbRollNode}" wrist_left_node="/${prefix}${WristLeftNode}" wrist_right_node="/${prefix}${WristRightNode}" wrist_pitch_calibration_angle="${WristPitchCalibrationAngle}" wrist_roll_calibration_angle="${WristRollCalibrationAngle}" />
+    <xacro:hand_mechanism mechanism_name="${prefix}Hand" serial_number="${hand_serial_number}" index_node="/${prefix}${IndexFingerNode}" middle_node="/${prefix}${MiddleFingerNode}" pinky_node="/${prefix}${PinkyFingerNode}" thumb_prox_node="/${prefix}${ThumbProximalNode}" thumb_dist_node="/${prefix}${ThumbDistalNode}" thumb_roll_node="/${prefix}${ThumbRollNode}" wrist_left_node="/${prefix}${WristLeftActuatorNode}" wrist_right_node="/${prefix}${WristRightActuatorNode}" wrist_pitch_calibration_angle="${WristPitchCalibrationAngle}" wrist_roll_calibration_angle="${WristRollCalibrationAngle}" />
     <xacro:hand_sensor_mechanism name="${prefix}HandSensors" serial_number="${hand_serial_number}_midas" node="/${prefix}${HandSensorNode}" />
     </Mechanisms>

File: instance/instances/robots/xacro/common/test_bench_template.xacro (robot description, xacro)
@@ -5,7 +5,6 @@
 	<xacro:include filename="../../../../../common/xacro/firmware/valkyrie_firmware.xacro"/>
 	<RobotInstance id="testbench" />
-	<Channels>
-	</Channels>
-	<!--<xacro:all_channels/>-->
+	<RobonetConfig>
+	</RobonetConfig>
     <xacro:firmware_base_url/>
 	<Mechanisms>

File: instance/instances/robots/xacro/common/valkyrie_full_template.xacro (robot description, xacro)
@@ -10,5 +10,5 @@
 	<xacro:include filename="../../../../../instance/instances/robots/xacro/common/joint_calibration_angles.xacro" />
 	<RobotInstance id="${instance}" />
-	<xacro:all_channels/>
+	<xacro:robonet_config/>
 	<Mechanisms>
 		<xacro:leg prefix="left" reflect="1" j1_serial_number="${leftLegJ1SerialNumber}" j2_serial_number="${leftLegJ2SerialNumber}" j3_serial_number="${leftLegJ3SerialNumber}" j4_serial_number="${leftLegJ4SerialNumber}" ankle_left_actuator_serial="${leftAnkleLeftActuatorSerialNumber}" ankle_right_actuator_serial="${leftAnkleRightActuatorSerialNumber}"/>

File: instance/instances/robots/xacro/limbs/arm/arm.xacro (robot description, xacro)
@@ -3,10 +3,10 @@
     <xacro:include filename="../../../../../../common/xacro/joint_names/valkyrie_joint_names.xacro"/>
     <xacro:macro name="arm" params="prefix reflect j1_serial_number j2_serial_number j3_serial_number j4_serial_number j5_serial_number forearm_serial_number" >
-    	<xacro:simple_mechanism name="${ShoulderPitchJointName}" serial_number="${j1_serial_number}" node="/trunk/${prefix}_arm_j1" calibration_angle="${ShoulderPitchCalibrationAngle}"/>
+        <xacro:simple_mechanism name="${ShoulderPitchJointName}" serial_number="${j1_serial_number}" node="/trunk/${prefix}${ShoulderPitchNode}" calibration_angle="${ShoulderPitchCalibrationAngle}"/>
     	<xacro:simple_mechanism name="${ShoulderRollJointName}" serial_number="${j2_serial_number}" node="/${prefix}${ShoulderRollNode}" calibration_angle="${reflect * -1.309}"/>
     	<xacro:simple_mechanism name="${ShoulderYawJointName}" serial_number="${j3_serial_number}" node="/${prefix}${ShoulderYawNode}" calibration_angle="${ShoulderYawCalibrationAngle}"/>
     	<xacro:simple_mechanism name="${ElbowPitchJointName}" serial_number="${j4_serial_number}" node="/${prefix}${ElbowPitchNode}" calibration_angle="${ElbowPitchCalibrationAngle}"/>
     	<xacro:simple_mechanism name="${ForearmYawJointName}" serial_number="${j5_serial_number}" node="/${prefix}${ForearmYawNode}" calibration_angle="${ForearmYawCalibrationAngle}"/>
-    	<xacro:hand_mechanism mechanism_name="${prefix}Hand" serial_number="${forearm_serial_number}" index_node="/${prefix}${IndexNode}" middle_node="/${prefix}${MiddleNode}" pinky_node="/${prefix}${PinkyNode}" thumb_prox_node="/${prefix}${ThumbProxNode}" thumb_dist_node="/${prefix}${ThumbDistNode}" thumb_roll_node="/${prefix}${ThumbRollNode}" wrist_left_node="/${prefix}${WristLeftNode}" wrist_right_node="/${prefix}${WristRightNode}" wrist_pitch_calibration_angle="${WristPitchCalibrationAngle}" wrist_roll_calibration_angle="${WristRollCalibrationAngle}" />
+    	<xacro:hand_mechanism mechanism_name="${prefix}Hand" serial_number="${forearm_serial_number}" index_node="/${prefix}${IndexFingerNode}" middle_node="/${prefix}${MiddleFingerNode}" pinky_node="/${prefix}${PinkyFingerNode}" thumb_prox_node="/${prefix}${ThumbProximalNode}" thumb_dist_node="/${prefix}${ThumbDistalNode}" thumb_roll_node="/${prefix}${ThumbRollNode}" wrist_left_node="/${prefix}${WristLeftActuatorNode}" wrist_right_node="/${prefix}${WristRightActuatorNode}" wrist_pitch_calibration_angle="${WristPitchCalibrationAngle}" wrist_roll_calibration_angle="${WristRollCalibrationAngle}" />
         <xacro:hand_sensor_mechanism name="${prefix}HandSensors" serial_number="${forearm_serial_number}_midas" node="/${prefix}${HandSensorNode}" />
     </xacro:macro>

File: instance/instances/robots/xacro/limbs/leg/leg.xacro (robot description, xacro)
@@ -3,5 +3,5 @@
     <xacro:include filename="../../../../../../common/xacro/joint_names/valkyrie_joint_names.xacro"/>
     <xacro:macro name="leg" params="prefix reflect j1_serial_number j2_serial_number j3_serial_number j4_serial_number ankle_left_actuator_serial ankle_right_actuator_serial" >
-    	<xacro:simple_mechanism name="${HipYawJointName}" serial_number="${j1_serial_number}" node="/pelvis/${prefix}_leg_j1" calibration_angle="${HipYawCalibrationAngle}"/>
+        <xacro:simple_mechanism name="${HipYawJointName}" serial_number="${j1_serial_number}" node="/pelvis/${prefix}${HipYawNode}" calibration_angle="${HipYawCalibrationAngle}"/>
     	<xacro:simple_mechanism name="${HipRollJointName}" serial_number="${j2_serial_number}" node="/${prefix}${HipRollNode}" calibration_angle="${HipRollCalibrationAngle}"/>
     	<xacro:simple_mechanism name="${HipPitchJointName}" serial_number="${j3_serial_number}" node="/${prefix}${HipPitchNode}" calibration_angle="${HipPitchCalibrationAngle}"/>
