Commit message: Remove use of prefix in nodes xacro

File: common/xacro/nodes/valkyrie_sim_nodes.xacro (robot description, xacro)
@@ -1,4 +1,3 @@
 <robot xmlns:xacro="http://www.ros.org/wiki/xacro" name="valkyrie_sim_nodes">
-	<!--<xacro:property name="HipYawNode" value="/pelvis/${prefix}_leg_j1" /> -->
 	<xacro:property name="TrunkYawNode" value="/pelvis/waist" /> <!--Yaw-->
 	<xacro:property name="LowerNeckPitchNode" value="/neck/j1" />
@@ -10,5 +9,5 @@
 	<xacro:property name="AnklePitchActuatorNode" value="_leg/ankle/pitch_actuator" />
 	<xacro:property name="AnkleRollActuatorNode" value="_leg/ankle/roll_actuator" />
-	<xacro:property name="ShoulderPitchNode" value="/trunk/${prefix}_arm_j1" />
+	<xacro:property name="ShoulderPitchNode" value="_arm_j1" />
 	<xacro:property name="ShoulderRollNode" value="_arm/j2" />
 	<xacro:property name="ShoulderYawNode" value="_arm/j3" />
@@ -19,6 +18,6 @@
 	<xacro:property name="WaistPitchActuatorNode" value="/trunk/pitch_actuator" /> <!--pitch-->
 	<xacro:property name="WaistRollActuatorNode" value="/trunk/roll_actuator" /> <!--roll-->
-	<xacro:property name="Athena1Node" value="/${prefix}_arm/athena1"/>
-	<xacro:property name="Athena2Node" value="/${prefix}_arm/athena2"/>
+	<xacro:property name="Athena1Node" value="_arm/athena1"/>
+	<xacro:property name="Athena2Node" value="_arm/athena2"/>
 	<xacro:property name="pelvis_middle_imu_node" value="/sensors/middlePelvisIMU" />
 	<xacro:property name="pelvis_rear_imu_node" value="/sensors/rearPelvisIMU" />
